Commit message: added different interfaces for motors

File: src/ballbot/bb_descrpition/urdf/bb.gazebo.xacro (robot description, xacro)
@@ -5,4 +5,5 @@
    <xacro:arg name="ground_truth" default="False" />
    <xacro:arg name="use_diff_drive" default="False" />
+   <xacro:arg name="motors_controller_type" default="EffortJointInterface" />
   <!-- controllers: -->
    <gazebo>
@@ -47,8 +48,8 @@
          <type>transmission_interface/SimpleTransmission</type>
          <joint name="wheel1_joint">
-            <hardwareInterface>hardware_interface/EffortJointInterface</hardwareInterface>
+            <hardwareInterface>hardware_interface/$(arg motors_controller_type)</hardwareInterface>
          </joint>
          <actuator name="wheel1_joint_actuator">
-            <hardwareInterface>hardware_interface/EffortJointInterface</hardwareInterface>
+            <hardwareInterface>hardware_interface/$(arg motors_controller_type)</hardwareInterface>
             <mechanicalReduction>1</mechanicalReduction>
          </actuator>
@@ -57,8 +58,8 @@
          <type>transmission_interface/SimpleTransmission</type>
          <joint name="wheel2_joint">
-            <hardwareInterface>hardware_interface/EffortJointInterface</hardwareInterface>
+            <hardwareInterface>hardware_interface/$(arg motors_controller_type)</hardwareInterface>
          </joint>
          <actuator name="wheel2_joint_actuator">
-            <hardwareInterface>hardware_interface/EffortJointInterface</hardwareInterface>
+            <hardwareInterface>hardware_interface/$(arg motors_controller_type)</hardwareInterface>
             <mechanicalReduction>1</mechanicalReduction>
          </actuator>
@@ -67,8 +68,8 @@
          <type>transmission_interface/SimpleTransmission</type>
          <joint name="wheel3_joint">
-            <hardwareInterface>hardware_interface/EffortJointInterface</hardwareInterface>
+            <hardwareInterface>hardware_interface/$(arg motors_controller_type)</hardwareInterface>
          </joint>
          <actuator name="wheel3_joint_actuator">
-            <hardwareInterface>hardware_interface/EffortJointInterface</hardwareInterface>
+            <hardwareInterface>hardware_interface/$(arg motors_controller_type)</hardwareInterface>
             <mechanicalReduction>1</mechanicalReduction>
          </actuator>
@@ -79,8 +80,8 @@
    <type>transmission_interface/SimpleTransmission</type>
    <joint name="subwheel${pos}_${orient}_joint">
-      <hardwareInterface>hardware_interface/EffortJointInterface</hardwareInterface>
+      <hardwareInterface>hardware_interface/$(arg motors_controller_type)</hardwareInterface>
    </joint>
    <actuator name="subwheel${pos}_${orient}_joint_actuator">
-      <hardwareInterface>hardware_interface/EffortJointInterface</hardwareInterface>
+      <hardwareInterface>hardware_interface/$(arg motors_controller_type)</hardwareInterface>
       <mechanicalReduction>1</mechanicalReduction>
    </actuator>
@@ -97,10 +98,12 @@
 </xacro:transmission_subwheel_macro>
 </xacro:macro>
-<xacro:transmission_subwheel_pos_macro pos="1">
+<!-- subwheels transmission's are not required or? (In case you  are not interested in the tf's of them -->
+<!-- generate subwheel transmission links: -->
+<!--<xacro:transmission_subwheel_pos_macro pos="1">
 </xacro:transmission_subwheel_pos_macro>
 <xacro:transmission_subwheel_pos_macro pos="2">
 </xacro:transmission_subwheel_pos_macro>
 <xacro:transmission_subwheel_pos_macro pos="3">
-</xacro:transmission_subwheel_pos_macro>
+</xacro:transmission_subwheel_pos_macro>-->
   <!-- </xacro:unless>-->
   <!-- p3d plugin (3D Position Interface for Ground Truth) -->
@@ -124,5 +127,5 @@
       <maxVel>0.01</maxVel>
       <minDepth>0</minDepth>
-      <mu1>0.0</mu1>
+      <mu1>0.0</mu1> <!-- das ist die Reibung am Boden oder?! -->
       <mu2>0.0</mu2>
       <fdir1>0 0 0</fdir1>

File: src/ballbot/bb_descrpition/urdf/bb.urdf.xacro (robot description, xacro)
@@ -20,9 +20,12 @@
     <xacro:property name="d_inertia_subwheel" value="0.00000001" />
     <!--motor values:-->
+    <!-- calculate max effort with emanual: http://support.robotis.com/en/product/actuator/dynamixel_x/xm_series/xm430-w350.htm -->
+    <!-- dynamixel: XM430-W350-T: see performance graph the effort depends on current, efficiency(E), torque : -->
+    <!-- http://simplemotor.com/calculations/ τ = (I * V * E *60) / (rpm * 2π) -->
    <xacro:property name="XL430_W250_max_effort" value="4.1" /> <!-- sollte: 1.5 -> klappt damit aber nicht. nimm 4.1 -->
    <xacro:property name="XL430_W250_max_velocity" value="5.7" /> <!-- sollte: ${61 * 2*pi/60}  klappt damit aber nicht nimm 5.7-->
-    <!-- trägheit des motors: -->
-   <xacro:property name="wheel_joint_damping" value="0.0" /> <!-- sollte: 0.5 -->
-   <xacro:property name="wheel_joint_friction" value="0.7" />  <!-- sollte: 1.0 -->
+    <!-- trägheit des motors: if these values are higher than the torques wheel does not turn, if this value is not small enough gazebo error-->
+   <xacro:property name="wheel_joint_damping" value="0.01" /> <!-- 0.01 sollte: 0.5 -->
+   <xacro:property name="wheel_joint_friction" value="0.05" />  <!-- 0.05 sollte: 1.0 -->
    <xacro:macro name="ballbot_macro">
       <link name="base_footprint" />
