Commit message: mit unseren stl files

File: src/ballbot/bb_descrpition/urdf/ball.gazebo.xacro (robot description, xacro)
@@ -13,60 +13,44 @@
       <maxContacts>10</maxContacts>
       <material>Gazebo/Grey</material>
-      <!--<collision name='ball_collision'>
-       <laser_retro>0</laser_retro>
-       <max_contacts>10</max_contacts>
-       <pose frame=''>0 0 0 0 -0 0</pose>
-       <geometry>
-       <mesh>
-         <uri>file://.../meshs/ball.stl</uri>
-         <scale>0.001 0.001 0.001</scale>
-       </mesh>
-       </geometry>
-       <surface>
-         <friction>
-           <ode>
-             <mu>0.5</mu>
-             <mu2>0.5</mu2>
-             <fdir1>0 0 0</fdir1>
-             <slip1>0</slip1>
-             <slip2>0</slip2>
-           </ode>
-           <torsional>
-             <coefficient>1</coefficient>
-             <patch_radius>0</patch_radius>
-             <surface_radius>0</surface_radius>
-             <use_patch_radius>1</use_patch_radius>
-             <ode>
-               <slip>0</slip>
-             </ode>
-           </torsional>
-         </friction>
-         <bounce>
-           <restitution_coefficient>0</restitution_coefficient>
-           <threshold>1e+06</threshold>
-         </bounce>
-         <contact>
-           <collide_without_contact>0</collide_without_contact>
-           <collide_without_contact_bitmask>1</collide_without_contact_bitmask>
-           <collide_bitmask>1</collide_bitmask>
-           <ode>
-             <soft_cfm>0</soft_cfm>
-             <soft_erp>0.2</soft_erp>
-             <kp>1e+13</kp>
-             <kd>1</kd>
-             <max_vel>0.01</max_vel>
-             <min_depth>0</min_depth>
-           </ode>
-           <bullet>
-             <split_impulse>1</split_impulse>
-             <split_impulse_penetration_threshold>-0.01</split_impulse_penetration_threshold>
-             <soft_cfm>0</soft_cfm>
-             <soft_erp>0.2</soft_erp>
-             <kp>1e+13</kp>
-             <kd>1</kd>
-           </bullet>
-         </contact>
-       </surface>
-     </collision>-->
+      <collision>
+         <surface>
+            <friction>
+               <torsional>
+                  <coefficient>1</coefficient>
+                  <patch_radius>0</patch_radius>
+                  <surface_radius>0</surface_radius>
+                  <use_patch_radius>1</use_patch_radius>
+                  <ode>
+                     <slip>0</slip>
+                  </ode>
+               </torsional>
+            </friction>
+            <bounce>
+               <restitution_coefficient>0</restitution_coefficient>
+               <threshold>1e+06</threshold>
+            </bounce>
+            <contact>
+               <collide_without_contact>0</collide_without_contact>
+               <collide_without_contact_bitmask>1</collide_without_contact_bitmask>
+               <collide_bitmask>1</collide_bitmask>
+               <ode>
+                  <soft_cfm>0</soft_cfm>
+                  <soft_erp>0.2</soft_erp>
+                  <kp>1e+13</kp>
+                  <kd>1</kd>
+                  <max_vel>0.01</max_vel>
+                  <min_depth>0</min_depth>
+               </ode>
+               <bullet>
+                  <split_impulse>1</split_impulse>
+                  <split_impulse_penetration_threshold>-0.01</split_impulse_penetration_threshold>
+                  <soft_cfm>0</soft_cfm>
+                  <soft_erp>0.2</soft_erp>
+                  <kp>1e+13</kp>
+                  <kd>1</kd>
+               </bullet>
+            </contact>
+         </surface>
+      </collision>
    </gazebo>
 </robot>

File: src/ballbot/bb_descrpition/urdf/ball.urdf.xacro (robot description, xacro)
@@ -7,5 +7,5 @@
          <parent link="base_footprint" />
          <child link="ball_link" />
-         <origin xyz="0.0 0.0 0.15" rpy="0.0 0.0 0.0" />
+         <origin xyz="0.0 0.0 0.070" rpy="0.0 0.0 0.0" />
       </joint>
       <link name="ball_link">
@@ -14,5 +14,5 @@
             <!-- 0.15?! -->
             <geometry>
-               <mesh filename="package://tuda_turtlebot3_description/meshes/base/ball.stl" scale="0.001 0.001 0.001" />
+               <mesh filename="package://tuda_turtlebot3_description/meshes/base/Kugel.stl" scale="0.001 0.001 0.001" />
             </geometry>
             <cast_shadows>1</cast_shadows>
@@ -22,5 +22,5 @@
          <inertial>
             <origin xyz="0.0 0.0 0.0" />
-            <mass value="1.34" />
+            <mass value="0.4" />
             <inertia ixx="0.0198384" ixy="0" ixz="0" iyy="0.0198384" iyz="0" izz="0.0198384" />
          </inertial>
@@ -28,5 +28,5 @@
             <origin xyz="0 0 0" rpy="0 0 0" />
             <geometry>
-               <mesh filename="package://tuda_turtlebot3_description/meshes/base/ball.stl" scale="0.001 0.001 0.001" />
+               <mesh filename="package://tuda_turtlebot3_description/meshes/base/Kugel.stl" scale="0.001 0.001 0.001" />
             </geometry>
          </collision>

File: src/ballbot/bb_descrpition/urdf/common_properties.xacro (robot description, xacro)
@@ -2,4 +2,5 @@
 <robot name="xacro_properties" xmlns:xacro="http://ros.org/wiki/xacro">
   <xacro:property name="M_PI" value="3.1415926535897931" />
+  <xacro:property name="grad_to_deg" value="0.01745329251" />
   <!-- Init colour -->
   <material name="black">

Commit message: added new omni wheel model, deleted hector stuff

File: src/ballbot/bb_descrpition/urdf/ball.gazebo.xacro (robot description, xacro)
@@ -13,5 +13,5 @@
       <maxContacts>10</maxContacts>
       <material>Gazebo/Grey</material>
-      <collision>
+<!--      <collision>
          <surface>
             <friction>
@@ -52,5 +52,5 @@
             </contact>
          </surface>
-      </collision>
+      </collision>-->
    </gazebo>
 </robot>

File: src/ballbot/bb_descrpition/urdf/ball.urdf.xacro (robot description, xacro)
@@ -1,5 +1,5 @@
 <?xml version="1.0" encoding="UTF-8"?>
 <robot xmlns:controller="http://playerstage.sourceforge.net/gazebo/xmlschema/#controller" xmlns:interface="http://ros.org/wiki/xacro" xmlns:sensor="http://playerstage.sourceforge.net/gazebo/xmlschema/#sensor" xmlns:xacro="http://ros.org/wiki/xacro" name="$(arg object_name)">
-   <xacro:include filename="$(find tuda_turtlebot3_description)/urdf/ball.gazebo.xacro" />
+   <xacro:include filename="$(find ballbot_description)/urdf/ball.gazebo.xacro" />
    <xacro:macro name="ball_macro">
       <link name="base_footprint" />
@@ -14,5 +14,5 @@
             <!-- 0.15?! -->
             <geometry>
-               <mesh filename="package://tuda_turtlebot3_description/meshes/base/Kugel.stl" scale="0.001 0.001 0.001" />
+               <mesh filename="package://ballbot_description/meshes/base/Kugel.stl" scale="0.001 0.001 0.001" />
             </geometry>
             <cast_shadows>1</cast_shadows>
@@ -28,5 +28,5 @@
             <origin xyz="0 0 0" rpy="0 0 0" />
             <geometry>
-               <mesh filename="package://tuda_turtlebot3_description/meshes/base/Kugel.stl" scale="0.001 0.001 0.001" />
+               <mesh filename="package://ballbot_description/meshes/base/Kugel.stl" scale="0.001 0.001 0.001" />
             </geometry>
          </collision>

File: src/ballbot/bb_descrpition/urdf/ball.xacro (robot description, xacro)
@@ -2,5 +2,5 @@
 <robot xmlns:xacro="http://ros.org/wiki/xacro" name="$(arg object_name)">
    <!-- einfach nur der Ball -->
-   <xacro:include filename="$(find tuda_turtlebot3_description)/urdf/ball.urdf.xacro" />
+   <xacro:include filename="$(find ballbot_description)/urdf/ball.urdf.xacro" />
    <xacro:ball_macro />
 </robot>

File: src/ballbot/bb_descrpition/urdf/bb.gazebo.xacro (robot description, xacro)
@@ -15,5 +15,32 @@
       </plugin>
    </gazebo>
-   <!--   The <transmission> element is used to link actuators to joints-->
+<!-- Skid steer drive controller
+<gazebo>
+  <plugin name="gazebo_ros_control" filename="libgazebo_ros_control.so" />
+  <plugin name="skid_steer_drive_controller" filename="libgazebo_ros_skid_steer_drive.so">
+    <alwaysOn>1</alwaysOn>
+    <updateRate>100.0</updateRate>
+    <robotNamespace>/</robotNamespace>
+    <leftFrontJoint>front_left_wheel_joint</leftFrontJoint>
+    <rightFrontJoint>front_right_wheel_joint</rightFrontJoint>
+    <leftRearJoint>back_left_wheel_joint</leftRearJoint>
+    <rightRearJoint>back_right_wheel_joint</rightRearJoint>
+    <wheelSeparation>${base_y_size}</wheelSeparation>
+    <wheelDiameter>${2*wheel_radius}</wheelDiameter>
+    <torque>100</torque>
+    <broadcastTF>1</broadcastTF>
+    <odometryFrame>map</odometryFrame>
+    <commandTopic>cmd_vel</commandTopic>
+    <odometryTopic>odom</odometryTopic>
+    <robotBaseFrame>base_footprint</robotBaseFrame>
+    <covariance_x>0.0001</covariance_x>
+    <covariance_y>0.0001</covariance_y>
+    <covariance_z>0.0001</covariance_z>
+    <covariance_yaw>0.0001</covariance_yaw>
+  </plugin>
+</gazebo>  -->
+   <!--   The <transmission> element is used to link actuators to joints
+          Without a transmission link there is no tf published!
+    -->
    <!--   <xacro:unless value="$(arg use_diff_drive)">-->
       <transmission name="wheel1_joint_transmission">
@@ -47,5 +74,45 @@
          </actuator>
       </transmission>
+<!-- subwheels transmission links: required for tf-->
+<xacro:macro name="transmission_subwheel_macro" params="pos orient">
+<transmission name="subwheel${pos}_${orient}_joint_transmission">
+   <type>transmission_interface/SimpleTransmission</type>
+   <joint name="subwheel${pos}_${orient}_joint">
+      <hardwareInterface>hardware_interface/EffortJointInterface</hardwareInterface>
+   </joint>
+   <actuator name="subwheel${pos}_${orient}_joint_actuator">
+      <hardwareInterface>hardware_interface/EffortJointInterface</hardwareInterface>
+      <mechanicalReduction>1</mechanicalReduction>
+   </actuator>
+</transmission>
+</xacro:macro>
+<xacro:macro name="transmission_subwheel_pos_macro" params="pos">
+<xacro:transmission_subwheel_macro pos="${pos}" orient="top">
+</xacro:transmission_subwheel_macro>
+<xacro:transmission_subwheel_macro pos="${pos}" orient="left">
+</xacro:transmission_subwheel_macro>
+<xacro:transmission_subwheel_macro pos="${pos}" orient="right">
+</xacro:transmission_subwheel_macro>
+<xacro:transmission_subwheel_macro pos="${pos}" orient="bottom">
+</xacro:transmission_subwheel_macro>
+</xacro:macro>
+<xacro:transmission_subwheel_pos_macro pos="1">
+</xacro:transmission_subwheel_pos_macro>
+<xacro:transmission_subwheel_pos_macro pos="2">
+</xacro:transmission_subwheel_pos_macro>
+<xacro:transmission_subwheel_pos_macro pos="3">
+</xacro:transmission_subwheel_pos_macro>
   <!-- </xacro:unless>-->
+  <!-- p3d plugin (3D Position Interface for Ground Truth) -->
+  <xacro:if value="$(arg ground_truth)">
+    <gazebo>
+      <plugin name="ground_truth" filename="libgazebo_ros_p3d.so">
+        <frameName>world</frameName>
+        <bodyName>base_footprint</bodyName>
+        <topicName>/gazebo/$(arg robot_name)/odom</topicName>
+        <updateRate>100.0</updateRate>
+      </plugin>
+    </gazebo>
+  </xacro:if>
    <!-- links: http://gazebosim.org/tutorials/?tut=ros_urdf-->
    <!--no multiple physics engines through urdf?!  -->
@@ -53,5 +120,5 @@
    <!--https://answers.ros.org/question/51956/simple-question-on-setting-bounce-properties-urdf/-->
    <gazebo reference="body_link">
-      <!-- shortforms: -->
+      <!-- shortforms:-->
       <gravity>1</gravity>
       <maxVel>0.01</maxVel>
@@ -66,5 +133,5 @@
       <laserRetro>0</laserRetro>
       <material>Gazebo/DarkGrey</material>
-      <!-- not available as short form - full sdf: -->
+      <!-- not available as short form - full sdf:
       <collision>
          <surface>
@@ -98,184 +165,113 @@
             </contact>
          </surface>
-      </collision>
+      </collision> -->
    </gazebo>
-   <gazebo reference="wheel1_link">
-      <gravity>1</gravity>
-      <maxVel>0.01</maxVel>
-      <minDepth>0</minDepth>
-      <mu1>0.2</mu1>
-      <mu2>0.0</mu2>
-      <fdir1>0 0 0</fdir1>
-      <kp>1e+13</kp>
-      <kd>1.0</kd>
-      <selfCollide>0</selfCollide>
-      <maxContacts>10</maxContacts>
-      <laserRetro>0</laserRetro>
-      <material>Gazebo/Orange</material>
-      <collision>
-         <surface>
-            <friction>
-               <torsional>
-                  <coefficient>0</coefficient>
-                  <patch_radius>0</patch_radius>
-                  <surface_radius>0</surface_radius>
-                  <use_patch_radius>0</use_patch_radius>
-                  <ode>
-                     <slip>0</slip>
-                  </ode>
-               </torsional>
-            </friction>
-            <bounce>
-               <restitution_coefficient>0</restitution_coefficient>
-               <threshold>1e+06</threshold>
-            </bounce>
-            <contact>
-               <collide_without_contact>0</collide_without_contact>
-               <collide_without_contact_bitmask>1</collide_without_contact_bitmask>
-               <collide_bitmask>1</collide_bitmask>
-               <ode>
-                  <soft_cfm>0</soft_cfm>
-                  <soft_erp>0.2</soft_erp>
-                  <kp>1e+13</kp>
-                  <kd>1</kd>
-                  <max_vel>0.01</max_vel>
-                  <min_depth>0</min_depth>
-               </ode>
-               <bullet>
-                 <split_impulse>1</split_impulse>
-                 <split_impulse_penetration_threshold>-0.01</split_impulse_penetration_threshold>
-                 <soft_cfm>0</soft_cfm>
-                 <soft_erp>0.2</soft_erp>
-                 <kp>1e+13</kp>
-                 <kd>1</kd>
-               </bullet>
-            </contact>
-         </surface>
-      </collision>
-   </gazebo>
-   <gazebo reference="wheel2_link">
-      <gravity>1</gravity>
-      <maxVel>0.01</maxVel>
-      <minDepth>0</minDepth>
-      <mu1>0.2</mu1>
-      <mu2>0.0</mu2>
-      <fdir1>0 0 0</fdir1>
-      <kp>1e+13</kp>
-      <kd>1.0</kd>
-      <selfCollide>0</selfCollide>
-      <maxContacts>10</maxContacts>
-      <laserRetro>0</laserRetro>
-      <material>Gazebo/Orange</material>
-      <collision>
-         <surface>
-            <friction>
-               <torsional>
-                  <coefficient>0</coefficient>
-                  <patch_radius>0</patch_radius>
-                  <surface_radius>0</surface_radius>
-                  <use_patch_radius>0</use_patch_radius>
-                  <ode>
-                     <slip>0</slip>
-                  </ode>
-               </torsional>
-            </friction>
-            <bounce>
-               <restitution_coefficient>0</restitution_coefficient>
-               <threshold>1e+06</threshold>
-            </bounce>
-            <contact>
-               <collide_without_contact>0</collide_without_contact>
-               <collide_without_contact_bitmask>1</collide_without_contact_bitmask>
-               <collide_bitmask>1</collide_bitmask>
-               <ode>
-                  <soft_cfm>0</soft_cfm>
-                  <soft_erp>0.2</soft_erp>
-                  <kp>1e+13</kp>
-                  <kd>1</kd>
-                  <max_vel>0.01</max_vel>
-                  <min_depth>0</min_depth>
-               </ode>
-               <bullet>
-                 <split_impulse>1</split_impulse>
-                 <split_impulse_penetration_threshold>-0.01</split_impulse_penetration_threshold>
-                 <soft_cfm>0</soft_cfm>
-                 <soft_erp>0.2</soft_erp>
-                 <kp>1e+13</kp>
-                 <kd>1</kd>
-               </bullet>
-            </contact>
-         </surface>
-      </collision>
-   </gazebo>
-   <gazebo reference="wheel3_link">
-      <gravity>1</gravity>
-      <maxVel>0.01</maxVel>
-      <minDepth>0</minDepth>
-      <mu1>0.2</mu1>
-      <mu2>0.0</mu2>
-      <fdir1>0 0 0</fdir1>
-      <kp>1e+13</kp>
-      <kd>1.0</kd>
-      <selfCollide>0</selfCollide>
-      <maxContacts>10</maxContacts>
-      <laserRetro>0</laserRetro>
-      <material>Gazebo/Orange</material>
-      <collision>
-         <surface>
-            <friction>
-               <torsional>
-                  <coefficient>0</coefficient>
-                  <patch_radius>0</patch_radius>
-                  <surface_radius>0</surface_radius>
-                  <use_patch_radius>0</use_patch_radius>
-                  <ode>
-                     <slip>0</slip>
-                  </ode>
-               </torsional>
-            </friction>
-            <bounce>
-               <restitution_coefficient>0</restitution_coefficient>
-               <threshold>1e+06</threshold>
-            </bounce>
-            <contact>
-               <collide_without_contact>0</collide_without_contact>
-               <collide_without_contact_bitmask>1</collide_without_contact_bitmask>
-               <collide_bitmask>1</collide_bitmask>
-               <ode>
-                  <soft_cfm>0</soft_cfm>
-                  <soft_erp>0.2</soft_erp>
-                  <kp>1e+13</kp>
-                  <kd>1</kd>
-                  <max_vel>0.01</max_vel>
-                  <min_depth>0</min_depth>
-               </ode>
-               <bullet>
-                 <split_impulse>1</split_impulse>
-                 <split_impulse_penetration_threshold>-0.01</split_impulse_penetration_threshold>
-                 <soft_cfm>0</soft_cfm>
-                 <soft_erp>0.2</soft_erp>
-                 <kp>1e+13</kp>
-                 <kd>1</kd>
-               </bullet>
-            </contact>
-         </surface>
-      </collision>
-   </gazebo>
+<!--  <gazebo reference="camera_mount_link">
+      <material>Gazebo/DarkGrey</material>
+  </gazebo>-->
+<!-- main wheels:
+mu: Friction coefficients μ for the principal contact directions along the contact surface
+kp: Contact stiffness for rigid body contacts
+kd: Contact damping k_d for rigid body contacts
+mu of speichen_wheel actually does not matter cause it has no contact point!
+-->
+<xacro:macro name="wheel" params="pos">
+<gazebo reference="wheel${pos}_link">
+<mu1>0</mu1>
+<mu2>0</mu2>
+<kp>500000.0</kp>
+<kd>10.0</kd>
+<minDepth>0.001</minDepth>
+<maxVel>0.1</maxVel>
+<fdir1>1 0 0</fdir1>
+<material>Gazebo/Orange</material>
+</gazebo>
+</xacro:macro>
+<xacro:wheel pos="1">
+</xacro:wheel>
+<xacro:wheel pos="2">
+</xacro:wheel>
+<xacro:wheel pos="3">
+</xacro:wheel>
+<!-- subwheels: -->
+<xacro:macro name="subwheel_params" params="suffix">
+<gazebo reference="subwheel${suffix}_link">
+<mu1>0.5</mu1>
+<mu2>0.5</mu2>
+<kp>500000.0</kp>
+<kd>100.0</kd>
+<minDepth>0.001</minDepth>
+<maxVel>0.1</maxVel>
+<fdir1>1 0 0</fdir1>
+<material>Gazebo/Green</material>
+</gazebo>
+</xacro:macro>
+<xacro:macro name="subwheel" params="pos">
+<xacro:subwheel_params suffix="${pos}_top">
+</xacro:subwheel_params>
+<xacro:subwheel_params suffix="${pos}_bottom">
+</xacro:subwheel_params>
+<xacro:subwheel_params suffix="${pos}_left">
+</xacro:subwheel_params>
+<xacro:subwheel_params suffix="${pos}_right">
+</xacro:subwheel_params>
+</xacro:macro>
+<xacro:subwheel pos="1">
+</xacro:subwheel>
+<xacro:subwheel pos="2">
+</xacro:subwheel>
+<xacro:subwheel pos="3">
+</xacro:subwheel>
+<xacro:subwheel pos="4">
+</xacro:subwheel>
    <!-- sensor links here! -->
 <gazebo reference="imu_link">
-  <sensor type="imu" name="imu">
+  <sensor name="imu" type="imu">
     <imu/>
-    <plugin name="imu_plugin" filename="libgazebo_ros_imu_sensor.so">
-      <robotNamespace></robotNamespace>
+    <plugin filename="libgazebo_ros_imu_sensor.so" name="imu_plugin">
+      <robotNamespace/>
       <frameName>imu_link</frameName>
       <topicName>/$(arg robot_name)/sensor/imu</topicName>
-      <updateRateHZ>200.0</updateRateHZ>
-      <gaussianNoise>0.0001</gaussianNoise>
+      <updateRateHZ>100.0</updateRateHZ>
+      <gaussianNoise>0.001</gaussianNoise>
       <xyzOffset>0.0 0.0 0.0</xyzOffset>
-      <!--<alwaysOn>True</alwaysOn>-->
-      <rpyOffset>0.0 0.0 ${pi}</rpyOffset>
+      <rpyOffset>0.0 0.0 0.0</rpyOffset>
     </plugin>
   </sensor>
 </gazebo>
+<gazebo reference="base_scan">
+   <material>Gazebo/Yellow</material>
+   <sensor name="lds_lfcd_sensor" type="ray">
+     <pose>0 0 0 0 0 0</pose>
+     <visualize>False</visualize>
+     <update_rate>5</update_rate>
+     <ray>
+       <scan>
+         <horizontal>
+           <samples>360</samples>
+           <resolution>1</resolution>
+           <min_angle>0.0</min_angle>
+           <max_angle>6.28</max_angle>
+         </horizontal>
+       </scan>
+       <range>
+         <min>0.120</min>
+         <max>3.5</max>
+         <resolution>0.015</resolution>
+       </range>
+       <noise>
+         <type>gaussian</type>
+         <mean>0.0</mean>
+         <stddev>0.01</stddev>
+       </noise>
+     </ray>
+     <plugin filename="libgazebo_ros_laser.so" name="gazebo_ros_lds_lfcd_controller">
+       <robotNamespace>/$(arg robot_name)/sensor</robotNamespace>
+       <topicName>scan_raw</topicName>
+       <frameName>base_scan</frameName>
+     </plugin>
+   </sensor>
+ </gazebo>
+<!-- real sense stuff in realsense_camera.urdf.xacro -->
   <!-- https://answers.ros.org/question/12430/modelling-sensorsimu-in-gazebo/ libgazebo_ros_imu.so-->
 </robot>
