Commit message: added new omni wheel model, deleted hector stuff

File: src/ballbot/bb_descrpition/urdf/bb.urdf.xacro (robot description, xacro)
@@ -1,24 +1,29 @@
 <?xml version="1.0" encoding="UTF-8"?>
-<!-- Meshes:
-realsense_mount.stl
-tuda_turtlebot3_base.stl
-tuda_turtlebot3_base_simple.stl (without upboard, inboards wholes etc.)
-ballbot_base.stl
-bb_wheel-->
-<!-- actually ball should not have joint!
-but if I delete that sim does not work!
--->
-<!-- Ballbot: https://bitbucket.org/osrf/gazebo/issues/2335/how-to-set-the-friction-of-ballbot-the -->
-<!-- table of names sdf->xacro: http://gazebosim.org/tutorials/?tut=ros_urdf-->
-<!-- https://answers.ros.org/question/51956/simple-question-on-setting-bounce-properties-urdf/ -->
-<!--URDF: Joint elements: and their childs etc.:
-http://wiki.ros.org/urdf/XML/joint-->
-<robot xmlns:controller="http://playerstage.sourceforge.net/gazebo/xmlschema/#controller" xmlns:interface="http://ros.org/wiki/xacro" xmlns:sensor="http://playerstage.sourceforge.net/gazebo/xmlschema/#sensor" xmlns:xacro="http://ros.org/wiki/xacro">
+<!--radspeiche: x,y,z Werte vom Michi direkt aus solid edge auslesen -->
+<robot xmlns:controller="http://playerstage.sourceforge.net/gazebo/xmlschema/#controller"
+       xmlns:interface="http://ros.org/wiki/xacro"
+       xmlns:sensor="http://playerstage.sourceforge.net/gazebo/xmlschema/#sensor"
+       xmlns:xacro="http://ros.org/wiki/xacro">
    <!-- inits colors &PI -->
-   <xacro:include filename="$(find tuda_turtlebot3_description)/urdf/common_properties.xacro" />
-   <xacro:include filename="$(find tuda_turtlebot3_description)/urdf/bb.gazebo.xacro" />
-   <!--  <xacro:include filename="$(find hector_sensors_description)/urdf/realsense_camera.urdf.xacro" />
-  <xacro:include filename="$(find hector_xacro_tools)/urdf/inertia_tensors.urdf.xacro" />-->
-   <xacro:macro name="turtlebot3_macro" params="with_arm">
+   <xacro:include filename="$(find ballbot_description)/urdf/common_properties.xacro" />
+   <xacro:include filename="$(find ballbot_description)/urdf/bb.gazebo.xacro" />
+   <!-- <xacro:include filename="$(find ballbot_description)/urdf/realsense_camera.urdf.xacro" />
+<xacro:include filename="$(find hector_xacro_tools)/urdf/inertia_tensors.urdf.xacro" />-->
+   <!-- some properties:
+   see: http://support.robotis.com/en/product/actuator/dynamixel_x/xm_series/xm430-w350.htm
+   Effort: 4.1N.m (at 12.0V, 2.3A)  Velocity: 57rpm (at 14.8V) (no load speed)   -->
+    <!-- speichen wheel parameter: -->
+   <xacro:property name="mass_wheel" value="0.030" />
+   <xacro:property name="d_inertia_wheel" value="0.00001" /> <!-- unit is kg m^2 diagonal inertia value for ixx,iyy,izz -->
+    <!-- subwheels parameters : -->
+    <xacro:property name="mass_subwheel" value="0.006" /> <!-- should be 4g -> but sim fails for that -->
+    <xacro:property name="d_inertia_subwheel" value="0.00000001" />
+    <!--motor values:-->
+   <xacro:property name="XL430_W250_max_effort" value="4.1" /> <!-- sollte: 1.5 -> klappt damit aber nicht. nimm 4.1 -->
+   <xacro:property name="XL430_W250_max_velocity" value="5.7" /> <!-- sollte: ${61 * 2*pi/60}  klappt damit aber nicht nimm 5.7-->
+    <!-- trägheit des motors: -->
+   <xacro:property name="wheel_joint_damping" value="0.0" /> <!-- sollte: 0.5 -->
+   <xacro:property name="wheel_joint_friction" value="0.7" />  <!-- sollte: 1.0 -->
+   <xacro:macro name="ballbot_macro">
       <link name="base_footprint" />
       <joint name="body_joint" type="fixed">
@@ -26,11 +31,11 @@
          <child link="body_link" />
          <!-- World KS to Oberbau KS: Messung: 101+140   Michi: ${0.1149+0.08901}-->
-         <origin xyz="0.0 0.0 ${0.101+0.140}" rpy="0.0 0.0 0.0" />
+         <origin xyz="0.0 0.0 ${0.101+0.140-0.021}" rpy="0.0 0.0 0.0" />
       </joint>
       <link name="body_link">
          <visual>
-            <origin xyz="0.0 0.0 0.0" rpy="${M_PI*0.5} 0.0  0.0" />
+            <origin xyz="0.0 0.0 0.0" rpy="0.0 0.0  0.0" />
             <geometry>
-               <mesh filename="package://tuda_turtlebot3_description/meshes/base/TUD_Ballbot_V1.0MS_ohne_Raeder.stl" scale="0.001 0.001 0.001" />
+               <mesh filename="package://ballbot_description/meshes/base/Ballbot_ohne_Raeder_V2.0MS.stl" scale="0.001 0.001 0.001" />
             </geometry>
             <cast_shadows>1</cast_shadows>
@@ -49,115 +54,163 @@
             </geometry>
 <!--            <geometry>
-               <mesh filename="package://tuda_turtlebot3_description/meshes/base/TUD_Ballbot_V1.0MS_ohne_Raeder.stl" scale="0.001 0.001 0.001" />
+               <mesh filename="package://ballbot_description/meshes/base/Ballbot_ohne_Raeder_V2.0MS.stl" scale="0.001 0.001 0.001" />
             </geometry>-->
          </collision>
       </link>
-      <joint name="wheel1_joint" type="continuous">
-         <parent link="body_link" />
-         <child link="wheel1_link" />
-         <origin xyz="${-0.05956*cos(grad_to_deg*30)} ${-0.05956*sin(grad_to_deg*30)} -0.08901" rpy="${0.9804+M_PI} ${-M_PI*0.125} ${-M_PI*0.5}" />
-         <!--(0.2817-0.3434)-->
-         <axis xyz="0 1 0" />
-         <limit effort="4.1" velocity="5.7" />
-         <!--see: http://support.robotis.com/en/product/actuator/dynamixel_x/xm_series/xm430-w350.htm
-         Effort: 4.1N.m (at 12.0V, 2.3A)  Velocity: 57rpm (at 14.8V) (no load speed) -->
-         <dynamics friction="0.7" damping="0.0" />
-      </joint>
-      <link name="wheel1_link">
-         <visual>
-            <origin xyz="0 0 0" rpy="0 0 0" />
-            <geometry>
-               <mesh filename="package://tuda_turtlebot3_description/meshes/wheels/wheel.stl" scale="0.001 0.001 0.001" />
-            </geometry>
-            <cast_shadows>1</cast_shadows>
-            <transparency>0</transparency>
-            <material name="light_black" />
-         </visual>
-         <inertial>
-            <origin xyz="0.0 0.0 0.0" />
-            <mass value="0.050" />
-            <inertia ixx="0.000023157" ixy="0" ixz="0" iyy="0.000023157" iyz="0" izz="0.000023157" />
-         </inertial>
-         <collision>
-            <origin xyz="0 0 0" rpy="0 0 0" />
-            <geometry>
-               <mesh filename="package://tuda_turtlebot3_description/meshes/wheels/wheel.stl" scale="0.001 0.001 0.001" />
-            </geometry>
-         </collision>
-      </link>
-      <joint name="wheel2_joint" type="continuous">
-         <parent link="body_link" />
-         <child link="wheel2_link" />
-         <origin xyz="0 0.05956 -0.08901" rpy="${2.1474+M_PI} -0.4183 0.5584" />
-         <axis xyz="0 1 0" />
-         <limit effort="4.1" velocity="5.7" />
-         <dynamics friction="0.7" damping="0.0" />
-      </joint>
-      <link name="wheel2_link">
-         <visual>
-            <origin xyz="0 0 0" rpy="0 0 0" />
-            <geometry>
-               <mesh filename="package://tuda_turtlebot3_description/meshes/wheels/wheel.stl" scale="0.001 0.001 0.001" />
-            </geometry>
-            <cast_shadows>1</cast_shadows>
-            <transparency>0</transparency>
-            <material name="light_black" />
-         </visual>
-         <inertial>
-            <origin xyz="0.0 0.0 0.0" />
-            <mass value="0.050" />
-            <inertia ixx="0.000023157" ixy="0" ixz="0" iyy="0.000023157" iyz="0" izz="0.000023157" />
-         </inertial>
-         <collision>
-            <origin xyz="0 0 0" rpy="0 0 0" />
-            <geometry>
-               <mesh filename="package://tuda_turtlebot3_description/meshes/wheels/wheel.stl" scale="0.001 0.001 0.001" />
-            </geometry>
-         </collision>
-      </link>
-      <joint name="wheel3_joint" type="continuous">
-         <parent link="body_link" />
-         <child link="wheel3_link" />
-         <origin xyz="${0.05956*cos(grad_to_deg*30)} ${-0.05956*sin(grad_to_deg*30)} -0.08901" rpy="-2.1612 ${M_PI*0.125} ${M_PI*0.5}" />
-         <axis xyz="0 1 0" />
-         <limit effort="4.1" velocity="5.7" />
-         <dynamics friction="0.7" damping="0.0" />
-         <!-- set damping to 0? -->
-      </joint>
-      <link name="wheel3_link">
-         <visual>
-            <origin xyz="0 0 0" rpy="0 0 0" />
-            <geometry>
-               <mesh filename="package://tuda_turtlebot3_description/meshes/wheels/wheel.stl" scale="0.001 0.001 0.001" />
-            </geometry>
-            <cast_shadows>1</cast_shadows>
-            <transparency>0</transparency>
-            <material name="light_black" />
-         </visual>
-         <inertial>
-            <origin xyz="0.0 0.0 0.0" />
-            <mass value="0.050" />
-            <inertia ixx="0.000023157" ixy="0" ixz="0" iyy="0.000023157" iyz="0" izz="0.000023157" />
-         </inertial>
-         <collision>
-            <origin xyz="0 0 0" rpy="0 0 0" />
-            <geometry>
-               <mesh filename="package://tuda_turtlebot3_description/meshes/wheels/wheel.stl" scale="0.001 0.001 0.001" />
-            </geometry>
-         </collision>
-      </link>
+<!-- generate wheels and their joints: -->
+<xacro:macro name="wheel_link_joint_macro" params="pos *joint_origin">
+<joint name="wheel${pos}_joint" type="continuous">
+   <parent link="body_link" />
+   <child link="wheel${pos}_link" />
+   <xacro:insert_block name="joint_origin" />
+   <axis xyz="1 0 0" />
+   <limit effort="${XL430_W250_max_effort}" velocity="${XL430_W250_max_effort}" />
+   <dynamics friction="${wheel_joint_friction}" damping="${wheel_joint_damping}" />
+</joint>
+<link name="wheel${pos}_link">
+   <visual>
+      <origin xyz="0 0 0" rpy="0 0 0" />
+      <geometry>
+         <mesh filename="package://ballbot_description/meshes/wheels/Speichen_Orientation_Test_4.stl" scale="0.001 0.001 0.001" />
+      </geometry>
+      <cast_shadows>1</cast_shadows>
+      <transparency>0</transparency>
+      <material name="light_black" />
+   </visual>
+   <inertial>
+      <origin xyz="0.0 0.0 0.0" />
+      <mass value="${mass_wheel}" />
+      <inertia ixx="${d_inertia_wheel}" ixy="0" ixz="0" iyy="${d_inertia_wheel}" iyz="0" izz="${d_inertia_wheel}" />
+   </inertial>
+   <collision>
+      <origin xyz="0 0 0" rpy="0 0 0" />
+      <geometry>
+         <mesh filename="package://ballbot_description/meshes/wheels/Speichen_Orientation_Test_4.stl" scale="0.001 0.001 0.001" />
+      </geometry>
+   </collision>
+</link>
+</xacro:macro>
+<xacro:wheel_link_joint_macro pos="1">
+   <origin xyz="0.00015 -0.05734 -0.06826" rpy="${0} ${M_PI/4} ${-M_PI/2}" />
+</xacro:wheel_link_joint_macro>
+<xacro:wheel_link_joint_macro pos="2">
+         <origin xyz="0.04936 0.02891 -0.06826" rpy="${0} ${M_PI/4} ${M_PI/6}" />
+</xacro:wheel_link_joint_macro>
+<xacro:wheel_link_joint_macro pos="3">
+   <origin xyz="-0.04936 0.02867 -0.06826" rpy="${0} ${M_PI/4} ${-M_PI/6*7}" />
+</xacro:wheel_link_joint_macro>
+<!-- generate subwheels and their joints:
+just their origin differs:
+-->
+<xacro:macro name="subwheel_link_joint_macro" params="pos orient *joint_origin_sub">
+<joint name="subwheel${pos}_${orient}_joint" type="continuous">
+   <parent link="wheel${pos}_link" />
+   <child link="subwheel${pos}_${orient}_link" />
+   <xacro:insert_block name="joint_origin_sub" />
+   <axis xyz="1 0 0" />
+   <limit effort="0" velocity="0" />
+   <dynamics friction="0" damping="0" />
+</joint>
+<link name="subwheel${pos}_${orient}_link">
+   <visual>
+      <origin xyz="0 0 0" rpy="0 0 0" />
+      <geometry>
+         <mesh filename="package://ballbot_description/meshes/wheels/Wheel_FreeWheel_V2.0.stl" scale="0.001 0.001 0.001" />
+      </geometry>
+   </visual>
+   <inertial>
+      <origin xyz="0.0 0.0 0.0" />
+      <mass value="${mass_subwheel}" />
+      <inertia ixx="${d_inertia_subwheel}" ixy="0" ixz="0" iyy="${d_inertia_subwheel}" iyz="0" izz="${d_inertia_subwheel}" />
+   </inertial>
+   <collision>
+      <origin xyz="0 0 0" rpy="0 0 0" />
+      <geometry>
+         <mesh filename="package://ballbot_description/meshes/wheels/Wheel_FreeWheel_V2.0.stl" scale="0.001 0.001 0.001" />
+      </geometry>
+   </collision>
+</link>
+</xacro:macro>
+<xacro:macro name="subwheel_generate_macro" params="pos">
+<xacro:subwheel_link_joint_macro pos="${pos}" orient="top">
+   <origin xyz="0.0125 0 -0.0234" rpy="${M_PI} ${0} ${-M_PI/2}" />
+</xacro:subwheel_link_joint_macro>
+<xacro:subwheel_link_joint_macro pos="${pos}" orient="bottom">
+   <origin xyz="0.0125 0 0.0234" rpy="${0} ${0} ${-M_PI/2}" />
+</xacro:subwheel_link_joint_macro>
+<xacro:subwheel_link_joint_macro pos="${pos}" orient="right">
+   <origin xyz="0.0125 0.0234 0" rpy="${0} ${-M_PI/2} ${-M_PI/2}" />
+</xacro:subwheel_link_joint_macro>
+<xacro:subwheel_link_joint_macro pos="${pos}" orient="left">
+   <origin xyz="0.0125 -0.0234 0" rpy="${0} ${M_PI/2} ${-M_PI/2}" />
+</xacro:subwheel_link_joint_macro>
+</xacro:macro>
+<xacro:subwheel_generate_macro pos="1">
+</xacro:subwheel_generate_macro>
+<xacro:subwheel_generate_macro pos="2">
+</xacro:subwheel_generate_macro>
+<xacro:subwheel_generate_macro pos="3">
+</xacro:subwheel_generate_macro>
       <!-- Ballbot Sensors-->
       <joint name="imu_joint" type="fixed">
          <parent link="body_link" />
          <child link="imu_link" />
-         <origin xyz="0 0 0.062" rpy="0.0 0.0 0" />
+         <origin xyz="0 0 0.068" rpy="0.0 0.0 0" />
       </joint>
       <link name="imu_link">
          <inertial>
             <origin xyz="0.0 0.0 0.0" />
-            <mass value="0.001" />
-            <inertia ixx="0.001" ixy="0.0" ixz="0.0" iyy="0.001" iyz="0.0" izz="0.001" />
+            <mass value="0.00001" />
+            <inertia ixx="0.00000001" ixy="0.0" ixz="0.0" iyy="0.00000001" iyz="0.0" izz="0.00000001" />
          </inertial>
       </link>
+<!--laser sensor: -->
+<joint name="scan_joint" type="fixed">
+  <parent link="body_link" />
+  <child link="base_scan" />
+  <origin xyz="0.02076 0 0.1225" rpy="0.0 0.0 0.0" />
+</joint>
+<link name="base_scan">
+  <inertial>
+    <mass value="0.00001" />
+   <!-- TODO origin here! -->
+    <origin xyz="-0.00687 0.0001 0.0038" />
+    <inertia ixx="-1.801e-06" ixy="-0.007e-06" ixz="3.231e-06"
+             iyy="-7.595e-06" iyz="0.004e-06"
+             izz="-5.794e-06" />
+  </inertial>
+</link>
+<!--
+<joint name="realsense_mount_joint" type="fixed">
+<parent link="body_link" />
+<child link="camera_mount_link" />
+<origin xyz="0.17407 -0.04586 0.03995" rpy="0.0 0.0 ${pi}" />
+</joint>
+<link name="camera_mount_link">
+<visual>
+<origin xyz="0.00133 -0.046 -0.00326" rpy="0.0 0.0 0.0" />
+<geometry>
+<mesh filename="package://ballbot_description/meshes/base/realsense_mount.stl" scale="0.001 0.001 0.001" />
+</geometry>
+<material name="dark" />
+</visual>
+<collision>
+<origin xyz="0.00133 -0.046 -0.00326" rpy="0.0 0.0 0.0" />
+<geometry>
+<box size="0.0175 0.134 0.024" />
+</geometry>
+</collision>
+<inertial>
+<mass value="0.023" />
+<origin xyz="0.00616 -0.04132 -0.00000235" />
+<inertia ixx="40.506e-06" ixy="-0.712e-06" ixz="0.472e-06"
+       iyy="2.546e-06" iyz="-0.601e-06"
+       izz="39.799e-06" />
+</inertial>
+</link>
+<xacro:realsense_camera name="camera" parent="camera_mount_link">
+<origin xyz="0.0 0.005 -0.00337" rpy="0.0 0.0 ${pi}" />
+</xacro:realsense_camera>
+-->
    </xacro:macro>
 </robot>

File: src/ballbot/bb_descrpition/urdf/bb.xacro (robot description, xacro)
@@ -1,10 +1,6 @@
 <?xml version="1.0" encoding="UTF-8"?>
 <robot xmlns:xacro="http://ros.org/wiki/xacro" name="$(arg robot_name)">
-   <!-- urdf.xacro's:
-bb.urdf.xacro
-tuda_turtlebot3.urdf.xacro-->
-   <xacro:include filename="$(find tuda_turtlebot3_description)/urdf/bb.urdf.xacro" />
-   <xacro:arg name="with_arm" default="False" />
-   <!-- Oberbau: -->
-   <xacro:turtlebot3_macro with_arm="$(arg with_arm)" />
+   <xacro:include filename="$(find ballbot_description)/urdf/bb.urdf.xacro" />
+    <!-- Exectue Macro for Ballbot: -->
+   <xacro:ballbot_macro/>
 </robot>

File: src/ballbot/bb_descrpition/urdf/common_properties.xacro (robot description, xacro)
@@ -2,5 +2,5 @@
 <robot name="xacro_properties" xmlns:xacro="http://ros.org/wiki/xacro">
   <xacro:property name="M_PI" value="3.1415926535897931" />
-  <xacro:property name="grad_to_deg" value="0.01745329251" />
+  <xacro:property name="deg_to_rad" value="0.01745329251" />
   <!-- Init colour -->
   <material name="black">

Commit message: white and yellow ball

File: src/ballbot/bb_descrpition/urdf/ball.gazebo.xacro (robot description, xacro)
@@ -12,5 +12,5 @@
       <selfCollide>0</selfCollide>
       <maxContacts>10</maxContacts>
-      <material>Gazebo/Grey</material>
+      <material>Gazebo/White</material>
 <!--      <collision>
          <surface>

File: src/ballbot/bb_descrpition/urdf/ball.urdf.xacro (robot description, xacro)
@@ -1,4 +1,7 @@
 <?xml version="1.0" encoding="UTF-8"?>
-<robot xmlns:controller="http://playerstage.sourceforge.net/gazebo/xmlschema/#controller" xmlns:interface="http://ros.org/wiki/xacro" xmlns:sensor="http://playerstage.sourceforge.net/gazebo/xmlschema/#sensor" xmlns:xacro="http://ros.org/wiki/xacro" name="$(arg object_name)">
+<robot xmlns:controller="http://playerstage.sourceforge.net/gazebo/xmlschema/#controller"
+       xmlns:interface="http://ros.org/wiki/xacro"
+       xmlns:sensor="http://playerstage.sourceforge.net/gazebo/xmlschema/#sensor"
+       xmlns:xacro="http://ros.org/wiki/xacro" name="$(arg ball_name)">
    <xacro:include filename="$(find ballbot_description)/urdf/ball.gazebo.xacro" />
    <xacro:macro name="ball_macro">

File: src/ballbot/bb_descrpition/urdf/ball.xacro (robot description, xacro)
@@ -1,6 +1,12 @@
 <?xml version="1.0" encoding="UTF-8"?>
-<robot xmlns:xacro="http://ros.org/wiki/xacro" name="$(arg object_name)">
-   <!-- einfach nur der Ball -->
-   <xacro:include filename="$(find ballbot_description)/urdf/ball.urdf.xacro" />
-   <xacro:ball_macro />
+<robot xmlns:xacro="http://ros.org/wiki/xacro" name="$(arg ball_name)">
+<xacro:arg name="wheel_type_single" default="True" />
+  <xacro:if value="$(arg wheel_type_single)">
+    <xacro:include filename="$(find ballbot_description)/urdf/ball.urdf.xacro" />
+    <xacro:ball_macro />
+  </xacro:if>
+  <xacro:unless value="$(arg wheel_type_single)">
+    <xacro:include filename="$(find ballbot_description)/urdf/ball_double_wheel.urdf.xacro" />
+    <xacro:ball_double_macro/>
+  </xacro:unless>
 </robot>

File: src/ballbot/bb_descrpition/urdf/bb.xacro (robot description, xacro)
@@ -1,6 +1,14 @@
 <?xml version="1.0" encoding="UTF-8"?>
 <robot xmlns:xacro="http://ros.org/wiki/xacro" name="$(arg robot_name)">
-   <xacro:include filename="$(find ballbot_description)/urdf/bb.urdf.xacro" />
+<xacro:arg name="wheel_type_single" default="True" />
+   <xacro:if value="$(arg wheel_type_single)">
+      <xacro:include filename="$(find ballbot_description)/urdf/bb.urdf.xacro" />
+      <!-- Exectue Macro for Ballbot: -->
+      <xacro:ballbot_macro/>
+   </xacro:if>
+  <xacro:unless value="$(arg wheel_type_single)">
+    <xacro:include filename="$(find ballbot_description)/urdf/bb.urdf_double_wheel.xacro" />
     <!-- Exectue Macro for Ballbot: -->
-   <xacro:ballbot_macro/>
+    <xacro:ballbot_double_macro/>
+  </xacro:unless>
 </robot>
