Commit message: yellow ball right rolles

File: src/ballbot/bb_descrpition/urdf/ball_double_wheel.urdf.xacro (robot description, xacro)
@@ -4,16 +4,15 @@
        xmlns:sensor="http://playerstage.sourceforge.net/gazebo/xmlschema/#sensor"
        xmlns:xacro="http://ros.org/wiki/xacro" name="$(arg ball_name)">
-   <xacro:include filename="$(find ballbot_description)/urdf/ball_double_wheel.gazebo.xacro" />
-   <xacro:macro name="ball_double_macro">
+<xacro:include filename="$(find ballbot_description)/urdf/ball_double_wheel.gazebo.xacro" />
+<xacro:macro name="ball_double_macro">
       <link name="base_footprint" />
       <joint name="body_joint" type="fixed">
          <parent link="base_footprint" />
          <child link="ball_link" />
-         <origin xyz="0.0 0.0 0.070" rpy="0.0 0.0 0.0" />
+         <origin xyz="0.0 0.0 0.080" rpy="0.0 0.0 0.0" />
       </joint>
       <link name="ball_link">
          <visual>
             <origin xyz="0 0 0.0" rpy="0 0 0" />
-            <!-- 0.15?! -->
             <geometry>
                <mesh filename="package://ballbot_description/meshes/base/Ball_160mm_2.stl" scale="0.001 0.001 0.001" />
@@ -21,10 +20,10 @@
             <cast_shadows>1</cast_shadows>
             <transparency>0</transparency>
-            <material name="light_black" />
+            <material name="yellow"/>
          </visual>
          <inertial>
             <origin xyz="0.0 0.0 0.0" />
             <mass value="0.326" />
-            <inertia ixx="0.00083" ixy="0" ixz="0" iyy="0.00083" iyz="0" izz="0.00083" />
+            <inertia ixx="0.00139093333333" ixy="0" ixz="0" iyy="0.00139093333333" iyz="0" izz="0.00139093333333" />
          </inertial>
          <collision>
@@ -37,2 +36,5 @@
    </xacro:macro>
 </robot>
+<!-- Notes:
+Inertia Calculation: http://hyperphysics.phy-astr.gsu.edu/hbase/isph.html
+-->

File: src/ballbot/bb_descrpition/urdf/bb.gazebo.xacro (robot description, xacro)
@@ -236,5 +236,5 @@
       <frameName>imu_link</frameName>
       <topicName>/$(arg robot_name)/sensor/imu</topicName>
-      <updateRateHZ>100.0</updateRateHZ>
+      <updateRateHZ>200.0</updateRateHZ>
       <gaussianNoise>0.001</gaussianNoise>
       <xyzOffset>0.0 0.0 0.0</xyzOffset>

File: src/ballbot/bb_descrpition/urdf/bb.urdf.xacro (robot description, xacro)
@@ -49,5 +49,5 @@
             <origin xyz="0.0 0.0 0.0" />
             <mass value="1.557" />
-            <inertia ixx="1.567" ixy="-0.003" ixz="-0.002" iyy="0.331" iyz="0.010" izz="1.565" /> <!-- km dm^2 -->
+            <inertia ixx="0.01567" ixy="-0.00003" ixz="-0.00002" iyy="0.00331" iyz="0.00010" izz="0.01565" /> <!-- km m^2 -->
          </inertial>
          <collision>

File: src/ballbot/bb_descrpition/urdf/bb.urdf_double_wheel.xacro (robot description, xacro)
@@ -6,5 +6,5 @@
    <!-- inits colors &PI -->
    <xacro:include filename="$(find ballbot_description)/urdf/common_properties.xacro" />
-   <xacro:include filename="$(find ballbot_description)/urdf/bb.gazebo_double_wheel.xacro" />
+   <xacro:include filename="$(find ballbot_description)/urdf/bb_double_wheel.gazebo.xacro" />
    <!-- <xacro:include filename="$(find ballbot_description)/urdf/realsense_camera.urdf.xacro" />
    <xacro:include filename="$(find hector_xacro_tools)/urdf/inertia_tensors.urdf.xacro" />-->
@@ -13,9 +13,9 @@
    Effort: 4.1N.m (at 12.0V, 2.3A)  Velocity: 57rpm (at 14.8V) (no load speed)   -->
     <!-- speichen wheel parameter: -->
-   <xacro:property name="mass_wheel" value="0.030" /> <!-- rad mit mitnehmer ohne motor und ohne kleine schwarze subwheels -->
+   <xacro:property name="mass_wheel" value="0.062" /> <!-- rad mit mitnehmer ohne motor und ohne kleine schwarze subwheels -->
    <xacro:property name="d_inertia_wheel" value="0.00001" /> <!-- unit is kg m^2 diagonal inertia value for ixx,iyy,izz -->
     <!-- subwheels parameters : -->
-    <xacro:property name="mass_subwheel" value="0.006" /> <!-- should be 4g -> but sim fails for that -->
-    <xacro:property name="d_inertia_subwheel" value="0.00000001" />
+    <xacro:property name="mass_subwheel" value="0.006" /> <!--  -->
+    <xacro:property name="d_inertia_subwheel" value="0.00000001" /> <!-- unit is kg m^2 diagonal inertia value for ixx,iyy,izz -->
     <!--motor values:-->
     <!-- calculate max effort with emanual: http://support.robotis.com/en/product/actuator/dynamixel_x/xm_series/xm430-w350.htm -->
@@ -32,6 +32,6 @@
          <parent link="base_footprint" />
          <child link="body_link" />
-         <!-- World KS to Oberbau KS: Messung: 101+140   Michi: ${0.1149+0.08901}-->
-         <origin xyz="0.0 0.0 ${0.101+0.140-0.021}" rpy="0.0 0.0 0.0" />
+         <!-- the height point is ballmiddle point to ball_link + diameter/2 -->
+         <origin xyz="0.0 0.0 ${0.216+0.04}" rpy="0.0 0.0 0.0" />
       </joint>
       <link name="body_link">
@@ -47,6 +47,6 @@
          <inertial>
             <origin xyz="0.0 0.0 0.0" />
-            <mass value="1.557" />
-            <inertia ixx="1.567" ixy="-0.003" ixz="-0.002" iyy="0.331" iyz="0.010" izz="1.565" /> <!-- km dm^2 -->
+            <mass value="1.625" />
+            <inertia ixx="0.01567" ixy="-0.00003" ixz="-0.00002" iyy="0.00331" iyz="0.00010" izz="0.01565" /> <!-- km m^2 -->
          </inertial>
          <collision>
@@ -60,5 +60,5 @@
          </collision>
       </link>
-<!-- generate wheels and their joints: -->
+<!-- macro for wheels and their joints: -->
 <xacro:macro name="wheel_link_joint_macro" params="pos *joint_origin">
 <joint name="wheel${pos}_joint" type="continuous">
@@ -103,6 +103,5 @@
    <origin xyz="-0.03662 -0.06343 -0.09097" rpy="${0} ${M_PI/4} ${-2*M_PI/3}" />
 </xacro:wheel_link_joint_macro>
-<!-- generate subwheels and their joints:
-just their origin differs:
+<!-- macro for sub_wheels and their joints: -->
 <xacro:macro name="subwheel_link_joint_macro" params="pos orient *joint_origin_sub">
 <joint name="subwheel${pos}_${orient}_joint" type="continuous">
@@ -118,5 +117,5 @@
       <origin xyz="0 0 0" rpy="0 0 0" />
       <geometry>
-         <mesh filename="package://ballbot_description/meshes/wheels/Wheel_FreeWheel_V2.0.stl" scale="0.001 0.001 0.001" />
+         <mesh filename="package://ballbot_description/meshes/wheels/Wheel2_wheel_rightOrient.stl" scale="0.001 0.001 0.001" />
       </geometry>
    </visual>
@@ -129,23 +128,43 @@
       <origin xyz="0 0 0" rpy="0 0 0" />
       <geometry>
-         <mesh filename="package://ballbot_description/meshes/wheels/Wheel_FreeWheel_V2.0.stl" scale="0.001 0.001 0.001" />
+         <mesh filename="package://ballbot_description/meshes/wheels/Wheel2_wheel_rightOrient.stl" scale="0.001 0.001 0.001" />
       </geometry>
    </collision>
 </link>
 </xacro:macro>
+<!-- subwheel macros -->
 <xacro:macro name="subwheel_generate_macro" params="pos">
-<xacro:subwheel_link_joint_macro pos="${pos}" orient="top">
-   <origin xyz="0.0125 0 -0.0234" rpy="${M_PI} ${0} ${-M_PI/2}" />
-</xacro:subwheel_link_joint_macro>
-<xacro:subwheel_link_joint_macro pos="${pos}" orient="bottom">
-   <origin xyz="0.0125 0 0.0234" rpy="${0} ${0} ${-M_PI/2}" />
-</xacro:subwheel_link_joint_macro>
-<xacro:subwheel_link_joint_macro pos="${pos}" orient="right">
-   <origin xyz="0.0125 0.0234 0" rpy="${0} ${-M_PI/2} ${-M_PI/2}" />
-</xacro:subwheel_link_joint_macro>
-<xacro:subwheel_link_joint_macro pos="${pos}" orient="left">
-   <origin xyz="0.0125 -0.0234 0" rpy="${0} ${M_PI/2} ${-M_PI/2}" />
+<xacro:subwheel_link_joint_macro pos="${pos}" orient="1_out">
+   <origin xyz="0.01375 0.0 -0.0235" rpy="${0.0} ${-M_PI} ${-M_PI/2}" />
+</xacro:subwheel_link_joint_macro>
+<xacro:subwheel_link_joint_macro pos="${pos}" orient="2_out">
+   <origin xyz="0.01375 0.02235 -0.00726" rpy="${0.0} ${2/5*M_PI} ${-M_PI/2}" />
+</xacro:subwheel_link_joint_macro>
+<xacro:subwheel_link_joint_macro pos="${pos}" orient="3_out">
+   <origin xyz="0.01375 -0.02235 -0.00726" rpy="${0.0} ${-2/5*M_PI} ${-M_PI/2}" />
+</xacro:subwheel_link_joint_macro>
+<xacro:subwheel_link_joint_macro pos="${pos}" orient="4_out">
+   <origin xyz="0.01375 0.01381 0.01901" rpy="${0.0} ${4/5*M_PI} ${-M_PI/2}" />
+</xacro:subwheel_link_joint_macro>
+<xacro:subwheel_link_joint_macro pos="${pos}" orient="5_out">
+   <origin xyz="0.01375 -0.01381 0.01901" rpy="${0.0} ${-4/5*M_PI} ${-M_PI/2}" />
+</xacro:subwheel_link_joint_macro>
+<xacro:subwheel_link_joint_macro pos="${pos}" orient="1_in">
+   <origin xyz="0.00125 0.0 0.0235" rpy="${0.0} ${-M_PI} ${-M_PI/2}" />
+</xacro:subwheel_link_joint_macro>
+<xacro:subwheel_link_joint_macro pos="${pos}" orient="2_in">
+   <origin xyz="0.00125 -0.02235 0.00726" rpy="${0.0} ${2/5*M_PI} ${-M_PI/2}" />
+</xacro:subwheel_link_joint_macro>
+<xacro:subwheel_link_joint_macro pos="${pos}" orient="3_in">
+   <origin xyz="0.00125 0.02235 0.00726" rpy="${0.0} ${-2/5*M_PI} ${-M_PI/2}" />
+</xacro:subwheel_link_joint_macro>
+<xacro:subwheel_link_joint_macro pos="${pos}" orient="4_in">
+   <origin xyz="0.00125 0.01381 -0.01901" rpy="${0.0} ${-4/5*M_PI} ${-M_PI/2}" />
+</xacro:subwheel_link_joint_macro>
+<xacro:subwheel_link_joint_macro pos="${pos}" orient="5_in">
+   <origin xyz="0.00125 -0.01381 -0.01901" rpy="${0.0} ${+4/5*M_PI} ${-M_PI/2}" />
 </xacro:subwheel_link_joint_macro>
 </xacro:macro>
+<!-- generate subwheel's -->
 <xacro:subwheel_generate_macro pos="1">
 </xacro:subwheel_generate_macro>
@@ -154,5 +173,4 @@
 <xacro:subwheel_generate_macro pos="3">
 </xacro:subwheel_generate_macro>
--->
       <!-- Ballbot Sensors-->
       <joint name="imu_joint" type="fixed">

File: src/ballbot/bb_descrpition/urdf/bb_double_wheel.gazebo.xacro (robot description, xacro)
@@ -129,5 +129,5 @@
 <maxVel>0.1</maxVel>
 <fdir1>1 0 0</fdir1>
-<material>Gazebo/Orange</material>
+<material>Gazebo/Grey</material>
 </gazebo>
 </xacro:macro>
@@ -146,23 +146,33 @@
 <maxVel>0.1</maxVel>
 <fdir1>1 0 0</fdir1>
-<material>Gazebo/Green</material>
+<material>Gazebo/DarkGrey</material>
 </gazebo>
 </xacro:macro>
 <xacro:macro name="subwheel" params="pos">
-<xacro:subwheel_params suffix="${pos}_top">
-</xacro:subwheel_params>
-<xacro:subwheel_params suffix="${pos}_bottom">
-</xacro:subwheel_params>
-<xacro:subwheel_params suffix="${pos}_left">
-</xacro:subwheel_params>
-<xacro:subwheel_params suffix="${pos}_right">
-</xacro:subwheel_params>
-</xacro:macro>
-<!-- generate subwheels
+<xacro:subwheel_params suffix="${pos}_1_out">
+</xacro:subwheel_params>
+<xacro:subwheel_params suffix="${pos}_2_out">
+</xacro:subwheel_params>
+<xacro:subwheel_params suffix="${pos}_3_out">
+</xacro:subwheel_params>
+<xacro:subwheel_params suffix="${pos}_4_out">
+</xacro:subwheel_params>
+<xacro:subwheel_params suffix="${pos}_5_out">
+</xacro:subwheel_params>
+<xacro:subwheel_params suffix="${pos}_1_in">
+</xacro:subwheel_params>
+<xacro:subwheel_params suffix="${pos}_2_in">
+</xacro:subwheel_params>
+<xacro:subwheel_params suffix="${pos}_3_in">
+</xacro:subwheel_params>
+<xacro:subwheel_params suffix="${pos}_4_in">
+</xacro:subwheel_params>
+<xacro:subwheel_params suffix="${pos}_5_in">
+</xacro:subwheel_params>
+</xacro:macro>
+<!-- generate subwheels -->
 <xacro:subwheel pos="1"> </xacro:subwheel>
 <xacro:subwheel pos="2"> </xacro:subwheel>
 <xacro:subwheel pos="3"> </xacro:subwheel>
-<xacro:subwheel pos="4"> </xacro:subwheel>
--->
    <!-- sensor links here! -->
 <gazebo reference="imu_link">

File: src/ballbot/bb_descrpition/urdf/common_properties.xacro (robot description, xacro)
@@ -34,3 +34,6 @@
     <color rgba="1.0 1.0 1.0 1.0"/>
   </material>
+  <material name="yellow">
+    <color rgba="1.0 1.0 0.0 1.0"/>
+  </material>
 </robot>

Commit message: added realsense and rviz_only_launch_file

File: src/ballbot/bb_descrpition/urdf/ball_double_wheel.urdf.xacro (robot description, xacro)
@@ -14,5 +14,5 @@
       <link name="ball_link">
          <visual name ="basket_ball">
-            <origin xyz="0 0 0.0" rpy="0 0 0" />
+            <origin xyz="0.0 0.0 0.0" rpy="0 0 0" />
             <geometry> <!-- if you wanna use no texture use:  <mesh filename="package://ballbot_description/meshes/base/Ball_160mm_2.stl" scale="0.001 0.001 0.001" /> -->
                <mesh filename="package://ballbot_gazebo/models/soccer_ball/meshes/ball.dae" scale="0.001 0.001 0.001" />

File: src/ballbot/bb_descrpition/urdf/bb.urdf_double_wheel.xacro (robot description, xacro)
@@ -7,6 +7,6 @@
    <xacro:include filename="$(find ballbot_description)/urdf/common_properties.xacro" />
    <xacro:include filename="$(find ballbot_description)/urdf/bb_double_wheel.gazebo.xacro" />
-   <!-- <xacro:include filename="$(find ballbot_description)/urdf/realsense_camera.urdf.xacro" />
-   <xacro:include filename="$(find hector_xacro_tools)/urdf/inertia_tensors.urdf.xacro" />-->
+   <xacro:include filename="$(find ballbot_description)/urdf/realsense_camera.urdf.xacro" />
+   <!--<xacro:include filename="$(find hector_xacro_tools)/urdf/inertia_tensors.urdf.xacro" />-->
    <!-- some properties:
    see: http://support.robotis.com/en/product/actuator/dynamixel_x/xm_series/xm430-w350.htm
@@ -37,5 +37,5 @@
          <child link="body_link" />
          <!-- the height point is ballmiddle point to ball_link + diameter/2 -->
-         <origin xyz="0.0 0.0 ${0.215+0.04}" rpy="0.0 0.0 0.0" />
+         <origin xyz="0.0 0.0 ${0.2122+0.04}" rpy="0.0 0.0 0.0" />
       </joint>
       <link name="body_link">
@@ -176,4 +176,5 @@
       <xacro:subwheel_generate_macro pos="3" />
       <!-- Ballbot Sensors-->
+      <!-- NOTE that the sensors are modeled weightless because the whole body contanins in it's inertias the weights of the sensors (camera, lds) -->
       <joint name="imu_joint" type="fixed">
          <parent link="body_link" />
@@ -184,5 +185,5 @@
          <inertial>
             <origin xyz="0.0 0.0 0.0" />
-            <mass value="0.00001" />
+            <mass value="0.001" />
             <inertia ixx="0.00000001" ixy="0.0" ixz="0.0" iyy="0.00000001" iyz="0.0" izz="0.00000001" />
          </inertial>
@@ -192,19 +193,32 @@
          <parent link="body_link" />
          <child link="base_scan" />
-         <origin xyz="0.02076 0 0.1225" rpy="0.0 0.0 0.0" />
+         <origin xyz="0.00894 0.0 0.175" rpy="0.0 0.0 0.0" /> <!-- Messung Michi -->
       </joint>
-      <link name="base_scan">
-         <inertial>
-            <mass value="0.00001" />
-            <!-- TODO origin here! -->
-            <origin xyz="-0.00687 0.0001 0.0038" />
-            <inertia ixx="-1.801e-06" ixy="-0.007e-06" ixz="3.231e-06" iyy="-7.595e-06" iyz="0.004e-06" izz="-5.794e-06" />
-         </inertial>
-      </link>
-      <!--
+<link name="base_scan">
+  <visual>
+    <origin xyz="0.0 0.0 -0.01" rpy="0.0 0.0 ${pi}" />
+    <geometry>
+      <mesh filename="package://ballbot_description/meshes/sensors/lds.stl" scale="0.001 0.001 0.001" />
+    </geometry>
+    <material name="dark" />
+  </visual>
+  <collision>
+    <origin xyz="0.012 0.0 -0.01" rpy="0.0 0.0 0.0" />
+    <geometry>
+      <cylinder length="0.040" radius="0.05" />
+    </geometry>
+  </collision>
+  <inertial>
+    <mass value="0.00001" />
+    <origin xyz="-0.0000687 0.000001 0.000038" />
+    <inertia ixx="-1.801e-09" ixy="-0.007e-09" ixz="3.231e-09"
+             iyy="-7.595e-09" iyz="0.004e-09"
+             izz="-5.794e-09" />
+  </inertial>
+</link>
 <joint name="realsense_mount_joint" type="fixed">
 <parent link="body_link" />
 <child link="camera_mount_link" />
-<origin xyz="0.17407 -0.04586 0.03995" rpy="0.0 0.0 ${pi}" />
+<origin xyz="0.081 -0.0461 0.15045" rpy="0.0 0.0 ${pi}" />
 </joint>
 <link name="camera_mount_link">
@@ -217,21 +231,21 @@
 </visual>
 <collision>
-<origin xyz="0.00133 -0.046 -0.00326" rpy="0.0 0.0 0.0" />
+<origin xyz="0.00133 -0.056 -0.00326" rpy="0.0 0.0 0.0" />
 <geometry>
-<box size="0.0175 0.134 0.024" />
+<box size="0.0175 0.154 0.024" />
 </geometry>
 </collision>
 <inertial>
-<mass value="0.023" />
-<origin xyz="0.00616 -0.04132 -0.00000235" />
-<inertia ixx="40.506e-06" ixy="-0.712e-06" ixz="0.472e-06"
-       iyy="2.546e-06" iyz="-0.601e-06"
-       izz="39.799e-06" />
+<mass value="0.0001" />
+<origin xyz="0.0000616 -0.0004132 -0.0000000235" />
+<inertia ixx="40.506e-09" ixy="-0.712e-09" ixz="0.472e-09"
+       iyy="2.546e-09" iyz="-0.601e-09"
+       izz="39.799e-09" />
 </inertial>
 </link>
+<!-- exectutes the macro in realsense_camera.urdf.xacro -->
 <xacro:realsense_camera name="camera" parent="camera_mount_link">
-<origin xyz="0.0 0.005 -0.00337" rpy="0.0 0.0 ${pi}" />
+  <origin xyz="0.0 0.005 -0.00337" rpy="0.0 0.0 ${pi}" />
 </xacro:realsense_camera>
--->
    </xacro:macro>
 </robot>

File: src/ballbot/bb_descrpition/urdf/bb_double_wheel.gazebo.xacro (robot description, xacro)
@@ -1,11 +1,12 @@
 <?xml version="1.0" encoding="UTF-8"?>
 <robot xmlns:xacro="http://ros.org/wiki/xacro">
-   <xacro:arg name="laser_visual" default="False" />
+   <xacro:arg name="motors_controller_type" default="EffortJointInterface" />
+   <xacro:arg name="imu_update_rate" default="100" />
+   <xacro:arg name="control_period" default="0.01" />
+    <!-- not used yet: -->
    <xacro:arg name="imu_visual" default="False" />
    <xacro:arg name="ground_truth" default="False" />
    <xacro:arg name="use_diff_drive" default="False" />
-   <xacro:arg name="motors_controller_type" default="EffortJointInterface" />
-   <xacro:arg name="imu_update_rate" default="100" />
-   <xacro:arg name="control_period" default="0.01" />
+   <xacro:arg name="laser_visual" default="False" /> <!-- is this used yet?! -->
    <!-- controllers: -->
    <gazebo>
@@ -116,7 +117,7 @@
       <material>Gazebo/DarkGrey</material>
    </gazebo>
-   <!--  <gazebo reference="camera_mount_link">
+  <gazebo reference="camera_mount_link">
       <material>Gazebo/DarkGrey</material>
-  </gazebo>-->
+  </gazebo>
 <!-- do i need this for ground friction?! -->
 <gazebo reference="base_footprint">
@@ -191,37 +192,37 @@
       </sensor>
    </gazebo>
-   <gazebo reference="base_scan">
-      <material>Gazebo/Yellow</material>
-      <sensor name="lds_lfcd_sensor" type="ray">
-         <pose>0 0 0 0 0 0</pose>
-         <visualize>False</visualize>
-         <update_rate>5</update_rate>
-         <ray>
-            <scan>
-               <horizontal>
-                  <samples>360</samples>
-                  <resolution>1</resolution>
-                  <min_angle>0.0</min_angle>
-                  <max_angle>6.28</max_angle>
-               </horizontal>
-            </scan>
-            <range>
-               <min>0.120</min>
-               <max>3.5</max>
-               <resolution>0.015</resolution>
-            </range>
-            <noise>
-               <type>gaussian</type>
-               <mean>0.0</mean>
-               <stddev>0.01</stddev>
-            </noise>
-         </ray>
-         <plugin filename="libgazebo_ros_laser.so" name="gazebo_ros_lds_lfcd_controller">
-            <robotNamespace>/$(arg robot_name)/sensor</robotNamespace>
-            <topicName>scan_raw</topicName>
-            <frameName>base_scan</frameName>
-         </plugin>
-      </sensor>
-   </gazebo>
+<gazebo reference="base_scan">
+  <material>Gazebo/DarkGrey</material>
+  <sensor type="ray" name="lds_lfcd_sensor">
+    <pose>0 0 0 0 0 0</pose>
+    <visualize>$(arg laser_visual)</visualize>
+    <update_rate>5</update_rate>
+    <ray>
+      <scan>
+        <horizontal>
+          <samples>360</samples>
+          <resolution>1</resolution>
+          <min_angle>0.0</min_angle>
+          <max_angle>6.28</max_angle>
+        </horizontal>
+      </scan>
+      <range>
+        <min>0.120</min>
+        <max>3.5</max>
+        <resolution>0.015</resolution>
+      </range>
+      <noise>
+        <type>gaussian</type>
+        <mean>0.0</mean>
+        <stddev>0.01</stddev>
+      </noise>
+    </ray>
+    <plugin name="gazebo_ros_lds_lfcd_controller" filename="libgazebo_ros_laser.so">
+      <robotNamespace>/$(arg robot_name)/sensor</robotNamespace>
+      <topicName>scan_raw</topicName>
+      <frameName>base_scan</frameName>
+    </plugin>
+  </sensor>
+</gazebo>
    <!-- real sense stuff in realsense_camera.urdf.xacro -->
    <!-- https://answers.ros.org/question/12430/modelling-sensorsimu-in-gazebo/ libgazebo_ros_imu.so-->

File: src/ballbot/bb_descrpition/urdf/realsense_camera.urdf.xacro (robot description, xacro)
@@ -23,7 +23,7 @@
       <link name="${name}_link">
         <inertial>
-          <mass value="0.200" />
+          <mass value="0.000200" />
           <origin xyz="0 0 0" rpy="0 0 0" />
-          <inertia ixx="5.8083e-4" ixy="0" ixz="0" iyy="3.0833e-5" iyz="0" izz="5.9083e-4" />
+          <inertia ixx="5.8083e-9" ixy="0" ixz="0" iyy="3.0833e-9" iyz="0" izz="5.9083e-9" />
         </inertial>
         <visual>
@@ -102,5 +102,5 @@
     </xacro:realsense_camera_model>
     <gazebo reference="${name}_link">
-      <sensor type="camera" name="${name}_color">
+      <sensor type="camera" name="${name}_rgb">
         <always_on>1</always_on>
         <update_rate>30</update_rate>
@@ -113,5 +113,5 @@
           </image>
           <clip>
-            <near>0.1</near>
+            <near>0.001</near>
             <far>100</far>
           </clip>
@@ -126,8 +126,8 @@
         </camera>
         <plugin name="${name}_camera_depth_controller" filename="libgazebo_ros_camera.so">
-          <robotNamespace>$(arg robot_name)/sensor/${name}/color</robotNamespace>
+          <robotNamespace>$(arg robot_name)/sensor/${name}/rgb</robotNamespace>
           <imageTopicName>image_raw</imageTopicName>
           <cameraInfoTopicName>camera_info</cameraInfoTopicName>
-          <frameName>${name}_color_optical_frame</frameName>
+          <frameName>${name}_rgb_optical_frame</frameName>
         </plugin>
       </sensor>
