Commit message: rviz working

File: src/ballbot/bb_descrpition/urdf/ball_double_wheel.gazebo.xacro (robot description, xacro)
@@ -5,12 +5,51 @@
       <maxVel>0.01</maxVel>
       <minDepth>0</minDepth>
-      <mu1>0.5</mu1>
-      <mu2>0.5</mu2>
+      <mu1>1000</mu1>
+      <mu2>1000</mu2>
       <fdir1>0 0 0</fdir1>
-      <kp>1e+13</kp>
-      <kd>1.0</kd>
+      <kp>5e+6</kp>
+      <kd>10.0</kd>
       <selfCollide>0</selfCollide>
       <maxContacts>10</maxContacts>
-      <material>Gazebo/Yellow</material>
+<!--      <visual name="basket_ball">
+      <cast_shadows>false</cast_shadows>
+      <geometry>
+      <sphere>
+        <radius>0.08</radius>
+      </sphere>
+      </geometry>
+        <material>
+          <script>
+            <uri>model://grey_wall/materials/scripts</uri>
+            <uri>model://grey_wall/materials/textures</uri>
+            <name>vrc/grey_wall</name>
+          </script>
+        </material>
+      </visual>-->
+<!--      <material>
+        <script>
+          <uri>model://arena_2017/materials/scripts</uri>
+          <uri>model://arena_2017/materials/textures</uri>
+          <name>arena_2017/FloorGrass</name>
+        </script>
+      </material>-->
+<!--<visual>
+  <material>
+    <ambient>0.19225 0.19225 0.19225 1.0</ambient>
+    <diffuse>0.50754 0.50754 0.50754 1.0</diffuse>
+    <specular>0.508273 0.508273 0.508273 1.0</specular>
+    <emissive>0.0 0.0 0.0 0.0</emissive>
+  </material>
+</visual>-->
+   </gazebo>
+<!-- p3d plugin (3D Position Interface for Ground Truth)
+     This is required only for rviz that the balllink tf is known! -->
+   <gazebo>
+      <plugin name="ground_truth" filename="libgazebo_ros_p3d.so">
+         <frameName>world</frameName>
+         <bodyName>ball_link</bodyName>
+         <topicName>/gazebo/$(arg ball_name)/odom</topicName>
+         <updateRate>110.0</updateRate>
+      </plugin>
    </gazebo>
 </robot>

File: src/ballbot/bb_descrpition/urdf/ball_double_wheel.urdf.xacro (robot description, xacro)
@@ -6,19 +6,19 @@
 <xacro:include filename="$(find ballbot_description)/urdf/ball_double_wheel.gazebo.xacro" />
 <xacro:macro name="ball_double_macro">
-      <link name="base_footprint" />
+<!--      <link name="base_footprint_ball" />
       <joint name="body_joint" type="fixed">
-         <parent link="base_footprint" />
+         <parent link="base_footprint_ball" />
          <child link="ball_link" />
          <origin xyz="0.0 0.0 0.080" rpy="0.0 0.0 0.0" />
-      </joint>
+      </joint>-->
       <link name="ball_link">
-         <visual>
+         <visual name ="basket_ball">
             <origin xyz="0 0 0.0" rpy="0 0 0" />
-            <geometry>
-               <mesh filename="package://ballbot_description/meshes/base/Ball_160mm_2.stl" scale="0.001 0.001 0.001" />
+            <geometry> <!-- if you wanna use no texture use:  <mesh filename="package://ballbot_description/meshes/base/Ball_160mm_2.stl" scale="0.001 0.001 0.001" /> -->
+               <mesh filename="package://ballbot_gazebo/models/soccer_ball/meshes/ball.dae" scale="0.001 0.001 0.001" />
             </geometry>
             <cast_shadows>1</cast_shadows>
             <transparency>0</transparency>
-            <material name="yellow"/>
+            <material name="basket_ball"/>
          </visual>
          <inertial>
@@ -30,5 +30,5 @@
             <origin xyz="0 0 0" rpy="0 0 0" />
             <geometry>
-               <mesh filename="package://ballbot_description/meshes/base/Ball_160mm_2.stl" scale="0.001 0.001 0.001" />
+               <mesh filename="package://ballbot_gazebo/models/soccer_ball/meshes/ball.dae" scale="0.001 0.001 0.001" />
             </geometry>
          </collision>

File: src/ballbot/bb_descrpition/urdf/bb.urdf_double_wheel.xacro (robot description, xacro)
@@ -1,7 +1,7 @@
 <?xml version="1.0" encoding="UTF-8"?>
 <robot xmlns:controller="http://playerstage.sourceforge.net/gazebo/xmlschema/#controller"
-       xmlns:interface="http://ros.org/wiki/xacro"
-       xmlns:sensor="http://playerstage.sourceforge.net/gazebo/xmlschema/#sensor"
-       xmlns:xacro="http://ros.org/wiki/xacro">
+        xmlns:interface="http://ros.org/wiki/xacro"
+        xmlns:sensor="http://playerstage.sourceforge.net/gazebo/xmlschema/#sensor"
+        xmlns:xacro="http://ros.org/wiki/xacro">
    <!-- inits colors &PI -->
    <xacro:include filename="$(find ballbot_description)/urdf/common_properties.xacro" />
@@ -12,19 +12,23 @@
    see: http://support.robotis.com/en/product/actuator/dynamixel_x/xm_series/xm430-w350.htm
    Effort: 4.1N.m (at 12.0V, 2.3A)  Velocity: 57rpm (at 14.8V) (no load speed)   -->
-    <!-- speichen wheel parameter: -->
-   <xacro:property name="mass_wheel" value="0.062" /> <!-- rad mit mitnehmer ohne motor und ohne kleine schwarze subwheels -->
-   <xacro:property name="d_inertia_wheel" value="0.00001" /> <!-- unit is kg m^2 diagonal inertia value for ixx,iyy,izz -->
-    <!-- subwheels parameters : -->
-    <xacro:property name="mass_subwheel" value="0.006" /> <!--  -->
-    <xacro:property name="d_inertia_subwheel" value="0.00000001" /> <!-- unit is kg m^2 diagonal inertia value for ixx,iyy,izz -->
-    <!--motor values:-->
-    <!-- calculate max effort with emanual: http://support.robotis.com/en/product/actuator/dynamixel_x/xm_series/xm430-w350.htm -->
-    <!-- dynamixel: XM430-W350-T: see performance graph the effort depends on current, efficiency(E), torque : -->
-    <!-- http://simplemotor.com/calculations/ τ = (I * V * E *60) / (rpm * 2π) -->
-   <xacro:property name="XL430_W250_max_effort" value="4.1" /> <!-- sollte: 1.5 -> klappt damit aber nicht. nimm 4.1 -->
-   <xacro:property name="XL430_W250_max_velocity" value="5.7" /> <!-- sollte: ${61 * 2*pi/60}  klappt damit aber nicht nimm 5.7-->
-    <!-- trägheit des motors: if these values are higher than the torques wheel does not turn, if this value is not small enough gazebo error-->
-   <xacro:property name="wheel_joint_damping" value="0.01" /> <!-- 0.01 sollte: 0.5 -->
-   <xacro:property name="wheel_joint_friction" value="0.05" />  <!-- 0.05 sollte: 1.0 -->
+   <!-- wheel parameter: h=2.5cm, r=3cm m=63g calculate inertia via: https://en.wikipedia.org/wiki/List_of_moments_of_inertia  -->
+   <xacro:property name="mass_wheel" value="0.063" />    <!-- rad mit mitnehmer ohne motor und ohne kleine schwarze subwheels -->
+   <xacro:property name="d_inertia_wheel_xx" value="2.75e-5" />    <!-- unit is kg m^2 diagonal inertia value for ixx -->
+   <xacro:property name="d_inertia_wheel_yy_zz" value="1.718e-5" />    <!-- unit is kg m^2 diagonal inertia value for iyy,izz -->
+   <!-- subwheels parameters : -->
+   <xacro:property name="mass_subwheel" value="0.006" />
+   <xacro:property name="d_inertia_subwheel" value="0.00000001" />    <!-- unit is kg m^2 diagonal inertia value for ixx,iyy,izz -->
+   <!--motor values:-->
+   <!-- calculate max effort with emanual: http://support.robotis.com/en/product/actuator/dynamixel_x/xm_series/xm430-w350.htm -->
+   <!-- dynamixel: XM430-W350-T: see performance graph the effort depends on current, efficiency(E), torque : -->
+   <!-- http://simplemotor.com/calculations/ τ = (I * V * E *60) / (rpm * 2π) -->
+   <xacro:property name="XL430_W250_max_effort" value="4.1" />    <!-- sollte: 1.5 -> klappt damit aber nicht. nimm 4.1 -->
+   <xacro:property name="XL430_W250_max_velocity" value="5.7" />  <!-- sollte: ${61 * 2*pi/60}  klappt damit aber nicht nimm 5.7-->
+   <!-- trägheit des motors: if these values are higher than the torques wheel does not turn, if this value is not small enough gazebo error-->
+   <!-- damping: is the damping force which is proportional to the velocity of the moving body [Nm*s/rad] -->
+   <!-- friction: The physical static friction value of the joint [Nm] -->
+   <!-- see: http://wiki.ros.org/urdf/XML/joint -->
+   <xacro:property name="wheel_joint_damping" value="0.01" />    <!-- 0.01 sollte: 0.5 -->
+   <xacro:property name="wheel_joint_friction" value="0.05" />     <!-- 0.05 sollte: 1.0 -->
    <xacro:macro name="ballbot_double_macro">
       <link name="base_footprint" />
@@ -33,5 +37,5 @@
          <child link="body_link" />
          <!-- the height point is ballmiddle point to ball_link + diameter/2 -->
-         <origin xyz="0.0 0.0 ${0.216+0.04}" rpy="0.0 0.0 0.0" />
+         <origin xyz="0.0 0.0 ${0.215+0.04}" rpy="0.0 0.0 0.0" />
       </joint>
       <link name="body_link">
@@ -46,12 +50,12 @@
          </visual>
          <inertial>
-            <origin xyz="0.0 0.0 0.0" />
-            <mass value="1.625" />
-            <inertia ixx="0.01567" ixy="-0.00003" ixz="-0.00002" iyy="0.00331" iyz="0.00010" izz="0.01565" /> <!-- km m^2 -->
+            <origin xyz="0.0 0.0 0.05" /> <!-- important: here you can set the center of mass position! -->
+            <mass value="1.572" />             <!-- eigentlich: ixx="0.1" ixy="0.001" ixz="0.002" iyy="0.099" iyz="0.00" izz="0.007" -->
+            <inertia ixx="0.1" ixy="0.00" ixz="0.00" iyy="0.1" iyz="0.00" izz="0.007" />
          </inertial>
          <collision>
             <origin xyz="0 0 ${0.048*2}" rpy="0 0 0" />
             <geometry>
-              <cylinder length="${0.048*4}" radius="0.078" />  <!-- geht von der mitte des zylinders aus! -->
+               <cylinder length="${0.048*4}" radius="0.078" /> <!-- geht von der mitte des zylinders aus! -->
             </geometry>
             <!-- <geometry>
@@ -60,117 +64,115 @@
          </collision>
       </link>
-<!-- macro for wheels and their joints: -->
-<xacro:macro name="wheel_link_joint_macro" params="pos *joint_origin">
-<joint name="wheel${pos}_joint" type="continuous">
-   <parent link="body_link" />
-   <child link="wheel${pos}_link" />
-   <xacro:insert_block name="joint_origin" />
-   <axis xyz="1 0 0" />
-   <limit effort="${XL430_W250_max_effort}" velocity="${XL430_W250_max_effort}" />
-   <dynamics friction="${wheel_joint_friction}" damping="${wheel_joint_damping}" />
-</joint>
-<link name="wheel${pos}_link">
-   <visual>
-      <origin xyz="0 0 0" rpy="0 0 0" />
-      <geometry>
-         <mesh filename="package://ballbot_description/meshes/wheels/Wheel2_Double_ohneRaeder.stl" scale="0.001 0.001 0.001" />
-      </geometry>
-      <cast_shadows>1</cast_shadows>
-      <transparency>0</transparency>
-      <material name="light_black" />
-   </visual>
-   <inertial>
-      <origin xyz="0.0 0.0 0.0" />
-      <mass value="${mass_wheel}" />
-      <inertia ixx="${d_inertia_wheel}" ixy="0" ixz="0" iyy="${d_inertia_wheel}" iyz="0" izz="${d_inertia_wheel}" />
-   </inertial>
-   <collision>
-      <origin xyz="0 0 0" rpy="0 0 0" />
-      <geometry>
-         <mesh filename="package://ballbot_description/meshes/wheels/Wheel2_Double_ohneRaeder.stl" scale="0.001 0.001 0.001" />
-      </geometry>
-   </collision>
-</link>
-</xacro:macro>
-<!-- generate wheels -->
-<xacro:wheel_link_joint_macro pos="1">
-   <origin xyz="0.07324 0.0 -0.09097" rpy="${0} ${M_PI/4} ${0}" /> <!-- Bezug immer auf Basis Koordinaten System , Basis ändert sich nie!-->
-</xacro:wheel_link_joint_macro>
-<xacro:wheel_link_joint_macro pos="2">
-   <origin xyz="-0.03662 +0.06343 -0.09097" rpy="${0} ${M_PI/4} ${+2*M_PI/3}" />
-</xacro:wheel_link_joint_macro>
-<xacro:wheel_link_joint_macro pos="3">
-   <origin xyz="-0.03662 -0.06343 -0.09097" rpy="${0} ${M_PI/4} ${-2*M_PI/3}" />
-</xacro:wheel_link_joint_macro>
-<!-- macro for sub_wheels and their joints: -->
-<xacro:macro name="subwheel_link_joint_macro" params="pos orient *joint_origin_sub">
-<joint name="subwheel${pos}_${orient}_joint" type="continuous">
-   <parent link="wheel${pos}_link" />
-   <child link="subwheel${pos}_${orient}_link" />
-   <xacro:insert_block name="joint_origin_sub" />
-   <axis xyz="1 0 0" />
-   <limit effort="0" velocity="0" />
-   <dynamics friction="0" damping="0" />
-</joint>
-<link name="subwheel${pos}_${orient}_link">
-   <visual>
-      <origin xyz="0 0 0" rpy="0 0 0" />
-      <geometry>
-         <mesh filename="package://ballbot_description/meshes/wheels/Wheel2_wheel_rightOrient.stl" scale="0.001 0.001 0.001" />
-      </geometry>
-   </visual>
-   <inertial>
-      <origin xyz="0.0 0.0 0.0" />
-      <mass value="${mass_subwheel}" />
-      <inertia ixx="${d_inertia_subwheel}" ixy="0" ixz="0" iyy="${d_inertia_subwheel}" iyz="0" izz="${d_inertia_subwheel}" />
-   </inertial>
-   <collision>
-      <origin xyz="0 0 0" rpy="0 0 0" />
-      <geometry>
-         <mesh filename="package://ballbot_description/meshes/wheels/Wheel2_wheel_rightOrient.stl" scale="0.001 0.001 0.001" />
-      </geometry>
-   </collision>
-</link>
-</xacro:macro>
-<!-- subwheel macros -->
-<xacro:macro name="subwheel_generate_macro" params="pos">
-<xacro:subwheel_link_joint_macro pos="${pos}" orient="1_out">
-   <origin xyz="0.01375 0.0 -0.0235" rpy="${0.0} ${-M_PI} ${-M_PI/2}" />
-</xacro:subwheel_link_joint_macro>
-<xacro:subwheel_link_joint_macro pos="${pos}" orient="2_out">
-   <origin xyz="0.01375 0.02235 -0.00726" rpy="${0.0} ${2/5*M_PI} ${-M_PI/2}" />
-</xacro:subwheel_link_joint_macro>
-<xacro:subwheel_link_joint_macro pos="${pos}" orient="3_out">
-   <origin xyz="0.01375 -0.02235 -0.00726" rpy="${0.0} ${-2/5*M_PI} ${-M_PI/2}" />
-</xacro:subwheel_link_joint_macro>
-<xacro:subwheel_link_joint_macro pos="${pos}" orient="4_out">
-   <origin xyz="0.01375 0.01381 0.01901" rpy="${0.0} ${4/5*M_PI} ${-M_PI/2}" />
-</xacro:subwheel_link_joint_macro>
-<xacro:subwheel_link_joint_macro pos="${pos}" orient="5_out">
-   <origin xyz="0.01375 -0.01381 0.01901" rpy="${0.0} ${-4/5*M_PI} ${-M_PI/2}" />
-</xacro:subwheel_link_joint_macro>
-<xacro:subwheel_link_joint_macro pos="${pos}" orient="1_in">
-   <origin xyz="0.00125 0.0 0.0235" rpy="${0.0} ${-M_PI} ${-M_PI/2}" />
-</xacro:subwheel_link_joint_macro>
-<xacro:subwheel_link_joint_macro pos="${pos}" orient="2_in">
-   <origin xyz="0.00125 -0.02235 0.00726" rpy="${0.0} ${2/5*M_PI} ${-M_PI/2}" />
-</xacro:subwheel_link_joint_macro>
-<xacro:subwheel_link_joint_macro pos="${pos}" orient="3_in">
-   <origin xyz="0.00125 0.02235 0.00726" rpy="${0.0} ${-2/5*M_PI} ${-M_PI/2}" />
-</xacro:subwheel_link_joint_macro>
-<xacro:subwheel_link_joint_macro pos="${pos}" orient="4_in">
-   <origin xyz="0.00125 0.01381 -0.01901" rpy="${0.0} ${-4/5*M_PI} ${-M_PI/2}" />
-</xacro:subwheel_link_joint_macro>
-<xacro:subwheel_link_joint_macro pos="${pos}" orient="5_in">
-   <origin xyz="0.00125 -0.01381 -0.01901" rpy="${0.0} ${+4/5*M_PI} ${-M_PI/2}" />
-</xacro:subwheel_link_joint_macro>
-</xacro:macro>
-<!-- generate subwheel's -->
-<xacro:subwheel_generate_macro pos="1">
-</xacro:subwheel_generate_macro>
-<xacro:subwheel_generate_macro pos="2">
-</xacro:subwheel_generate_macro>
-<xacro:subwheel_generate_macro pos="3">
-</xacro:subwheel_generate_macro>
+      <!-- macro for wheels and their joints: -->
+      <xacro:macro name="wheel_link_joint_macro" params="pos *joint_origin">
+         <joint name="wheel${pos}_joint" type="continuous">
+            <parent link="body_link" />
+            <child link="wheel${pos}_link" />
+            <xacro:insert_block name="joint_origin" />
+            <axis xyz="1 0 0" />
+            <limit effort="${XL430_W250_max_effort}" velocity="${XL430_W250_max_effort}" />
+            <dynamics friction="${wheel_joint_friction}" damping="${wheel_joint_damping}" />
+         </joint>
+         <link name="wheel${pos}_link">
+            <visual>
+               <origin xyz="0 0 0" rpy="0 0 0" />
+               <geometry>
+                  <mesh filename="package://ballbot_description/meshes/wheels/Wheel2_Double_ohneRaeder.stl" scale="0.001 0.001 0.001" />
+               </geometry>
+               <cast_shadows>1</cast_shadows>
+               <transparency>0</transparency>
+               <material name="light_black" />
+            </visual>
+            <inertial>
+               <origin xyz="0.0 0.0 0.0" />
+               <mass value="${mass_wheel}" />
+               <inertia ixx="${d_inertia_wheel_xx}" ixy="0.0" ixz="0.0" iyy="${d_inertia_wheel_yy_zz}" iyz="0.0" izz="${d_inertia_wheel_yy_zz}" />
+            </inertial>
+            <collision>
+               <origin xyz="0 0 0" rpy="0 0 0" />
+               <geometry>
+                  <mesh filename="package://ballbot_description/meshes/wheels/Wheel2_Double_ohneRaeder.stl" scale="0.001 0.001 0.001" />
+               </geometry>
+            </collision>
+         </link>
+      </xacro:macro>
+      <!-- generate wheels -->
+      <!-- Bezug immer auf Basis Koordinaten System , Basis ändert sich nie!-->
+      <xacro:wheel_link_joint_macro pos="1">
+         <origin xyz="0.07324 0.0 -0.09097" rpy="${0} ${M_PI/4} ${0}" />
+      </xacro:wheel_link_joint_macro>
+      <xacro:wheel_link_joint_macro pos="2">
+         <origin xyz="-0.03662 +0.06343 -0.09097" rpy="${0} ${M_PI/4} ${+2*M_PI/3}" />
+      </xacro:wheel_link_joint_macro>
+      <xacro:wheel_link_joint_macro pos="3">
+         <origin xyz="-0.03662 -0.06343 -0.09097" rpy="${0} ${M_PI/4} ${-2*M_PI/3}" />
+      </xacro:wheel_link_joint_macro>
+      <!-- macro for sub_wheels and their joints: -->
+      <xacro:macro name="subwheel_link_joint_macro" params="pos orient *joint_origin_sub">
+         <joint name="subwheel${pos}_${orient}_joint" type="continuous">
+            <parent link="wheel${pos}_link" />
+            <child link="subwheel${pos}_${orient}_link" />
+            <xacro:insert_block name="joint_origin_sub" />
+            <axis xyz="1 0 0" />
+            <limit effort="0" velocity="0" />
+            <dynamics friction="0.0" damping="0.0" />
+         </joint>
+         <link name="subwheel${pos}_${orient}_link">
+            <visual>
+               <origin xyz="0 0 0" rpy="0 0 0" />
+               <geometry>
+                  <mesh filename="package://ballbot_description/meshes/wheels/Wheel2_wheel_rightOrient.stl" scale="0.001 0.001 0.001" />
+               </geometry>
+            </visual>
+            <inertial>
+               <origin xyz="0.0 0.0 0.0" />
+               <mass value="${mass_subwheel}" />
+               <inertia ixx="${d_inertia_subwheel}" ixy="0" ixz="0" iyy="${d_inertia_subwheel}" iyz="0" izz="${d_inertia_subwheel}" />
+            </inertial>
+            <collision>
+               <origin xyz="0 0 0" rpy="0 0 0" />
+               <geometry>
+                  <mesh filename="package://ballbot_description/meshes/wheels/Wheel2_wheel_rightOrient.stl" scale="0.001 0.001 0.001" />
+               </geometry>
+            </collision>
+         </link>
+      </xacro:macro>
+      <!-- subwheel macros -->
+      <xacro:macro name="subwheel_generate_macro" params="pos">
+         <xacro:subwheel_link_joint_macro pos="${pos}" orient="1_out">
+            <origin xyz="0.01375 0.0 -0.0235" rpy="${0.0} ${-M_PI} ${-M_PI/2}" />
+         </xacro:subwheel_link_joint_macro>
+         <xacro:subwheel_link_joint_macro pos="${pos}" orient="2_out">
+            <origin xyz="0.01375 0.02235 -0.00726" rpy="${0.0} ${2/5*M_PI} ${-M_PI/2}" />
+         </xacro:subwheel_link_joint_macro>
+         <xacro:subwheel_link_joint_macro pos="${pos}" orient="3_out">
+            <origin xyz="0.01375 -0.02235 -0.00726" rpy="${0.0} ${-2/5*M_PI} ${-M_PI/2}" />
+         </xacro:subwheel_link_joint_macro>
+         <xacro:subwheel_link_joint_macro pos="${pos}" orient="4_out">
+            <origin xyz="0.01375 0.01381 0.01901" rpy="${0.0} ${4/5*M_PI} ${-M_PI/2}" />
+         </xacro:subwheel_link_joint_macro>
+         <xacro:subwheel_link_joint_macro pos="${pos}" orient="5_out">
+            <origin xyz="0.01375 -0.01381 0.01901" rpy="${0.0} ${-4/5*M_PI} ${-M_PI/2}" />
+         </xacro:subwheel_link_joint_macro>
+         <xacro:subwheel_link_joint_macro pos="${pos}" orient="1_in">
+            <origin xyz="0.00125 0.0 0.0235" rpy="${0.0} ${-M_PI} ${-M_PI/2}" />
+         </xacro:subwheel_link_joint_macro>
+         <xacro:subwheel_link_joint_macro pos="${pos}" orient="2_in">
+            <origin xyz="0.00125 -0.02235 0.00726" rpy="${0.0} ${2/5*M_PI} ${-M_PI/2}" />
+         </xacro:subwheel_link_joint_macro>
+         <xacro:subwheel_link_joint_macro pos="${pos}" orient="3_in">
+            <origin xyz="0.00125 0.02235 0.00726" rpy="${0.0} ${-2/5*M_PI} ${-M_PI/2}" />
+         </xacro:subwheel_link_joint_macro>
+         <xacro:subwheel_link_joint_macro pos="${pos}" orient="4_in">
+            <origin xyz="0.00125 0.01381 -0.01901" rpy="${0.0} ${-4/5*M_PI} ${-M_PI/2}" />
+         </xacro:subwheel_link_joint_macro>
+         <xacro:subwheel_link_joint_macro pos="${pos}" orient="5_in">
+            <origin xyz="0.00125 -0.01381 -0.01901" rpy="${0.0} ${+4/5*M_PI} ${-M_PI/2}" />
+         </xacro:subwheel_link_joint_macro>
+      </xacro:macro>
+      <!-- generate subwheel's -->
+      <xacro:subwheel_generate_macro pos="1" />
+      <xacro:subwheel_generate_macro pos="2" />
+      <xacro:subwheel_generate_macro pos="3" />
       <!-- Ballbot Sensors-->
       <joint name="imu_joint" type="fixed">
@@ -186,21 +188,19 @@
          </inertial>
       </link>
-<!--laser sensor: -->
-<joint name="scan_joint" type="fixed">
-  <parent link="body_link" />
-  <child link="base_scan" />
-  <origin xyz="0.02076 0 0.1225" rpy="0.0 0.0 0.0" />
-</joint>
-<link name="base_scan">
-  <inertial>
-    <mass value="0.00001" />
-   <!-- TODO origin here! -->
-    <origin xyz="-0.00687 0.0001 0.0038" />
-    <inertia ixx="-1.801e-06" ixy="-0.007e-06" ixz="3.231e-06"
-             iyy="-7.595e-06" iyz="0.004e-06"
-             izz="-5.794e-06" />
-  </inertial>
-</link>
-<!--
+      <!--laser sensor: -->
+      <joint name="scan_joint" type="fixed">
+         <parent link="body_link" />
+         <child link="base_scan" />
+         <origin xyz="0.02076 0 0.1225" rpy="0.0 0.0 0.0" />
+      </joint>
+      <link name="base_scan">
+         <inertial>
+            <mass value="0.00001" />
+            <!-- TODO origin here! -->
+            <origin xyz="-0.00687 0.0001 0.0038" />
+            <inertia ixx="-1.801e-06" ixy="-0.007e-06" ixz="3.231e-06" iyy="-7.595e-06" iyz="0.004e-06" izz="-5.794e-06" />
+         </inertial>
+      </link>
+      <!--
 <joint name="realsense_mount_joint" type="fixed">
 <parent link="body_link" />

File: src/ballbot/bb_descrpition/urdf/bb.xacro (robot description, xacro)
@@ -1,5 +1,4 @@
 <?xml version="1.0" encoding="UTF-8"?>
 <robot xmlns:xacro="http://ros.org/wiki/xacro" name="$(arg robot_name)">
-<xacro:arg name="wheel_type_single" default="True" />
    <xacro:if value="$(arg wheel_type_single)">
       <xacro:include filename="$(find ballbot_description)/urdf/bb.urdf.xacro" />
