Commit message: rviz working

File: src/ballbot/bb_descrpition/urdf/bb_double_wheel.gazebo.xacro (robot description, xacro)
@@ -6,12 +6,15 @@
    <xacro:arg name="use_diff_drive" default="False" />
    <xacro:arg name="motors_controller_type" default="EffortJointInterface" />
-  <!-- controllers: -->
+   <xacro:arg name="imu_update_rate" default="100" />
+   <xacro:arg name="control_period" default="0.01" />
+   <!-- controllers: -->
    <gazebo>
-     <!--Plugin loads hardware interfaces and controller manager -->
+      <!--Plugin loads hardware interfaces and controller manager -->
       <plugin name="gazebo_ros_control" filename="libgazebo_ros_control.so">
          <robotNamespace>/$(arg robot_name)/joints</robotNamespace>
          <robotParam>/$(arg robot_name)/robot_description</robotParam>
          <robotSimType>gazebo_ros_control/DefaultRobotHWSim</robotSimType>
-         <!--<controlPeriod> </controlPeriod>-->
+         <controlPeriod>$(arg control_period)</controlPeriod>
+         <!-- 100Hz means 0.01 control Period -->
       </plugin>
    </gazebo>
@@ -19,77 +22,79 @@
           Without a transmission link there is no tf published!
     -->
-      <transmission name="wheel1_joint_transmission">
+   <transmission name="wheel1_joint_transmission">
+      <type>transmission_interface/SimpleTransmission</type>
+      <joint name="wheel1_joint">
+         <hardwareInterface>hardware_interface/$(arg motors_controller_type)</hardwareInterface>
+      </joint>
+      <actuator name="wheel1_joint_actuator">
+         <hardwareInterface>hardware_interface/$(arg motors_controller_type)</hardwareInterface>
+         <mechanicalReduction>1</mechanicalReduction>
+      </actuator>
+   </transmission>
+   <transmission name="wheel2_joint_transmission">
+      <type>transmission_interface/SimpleTransmission</type>
+      <joint name="wheel2_joint">
+         <hardwareInterface>hardware_interface/$(arg motors_controller_type)</hardwareInterface>
+      </joint>
+      <actuator name="wheel2_joint_actuator">
+         <hardwareInterface>hardware_interface/$(arg motors_controller_type)</hardwareInterface>
+         <mechanicalReduction>1</mechanicalReduction>
+      </actuator>
+   </transmission>
+   <transmission name="wheel3_joint_transmission">
+      <type>transmission_interface/SimpleTransmission</type>
+      <joint name="wheel3_joint">
+         <hardwareInterface>hardware_interface/$(arg motors_controller_type)</hardwareInterface>
+      </joint>
+      <actuator name="wheel3_joint_actuator">
+         <hardwareInterface>hardware_interface/$(arg motors_controller_type)</hardwareInterface>
+         <mechanicalReduction>1</mechanicalReduction>
+      </actuator>
+   </transmission>
+   <!-- subwheels transmission links: required for tf-->
+   <xacro:macro name="transmission_subwheel_macro" params="pos orient">
+      <transmission name="subwheel${pos}_${orient}_joint_transmission">
          <type>transmission_interface/SimpleTransmission</type>
-         <joint name="wheel1_joint">
+         <joint name="subwheel${pos}_${orient}_joint">
             <hardwareInterface>hardware_interface/$(arg motors_controller_type)</hardwareInterface>
          </joint>
-         <actuator name="wheel1_joint_actuator">
+         <actuator name="subwheel${pos}_${orient}_joint_actuator">
             <hardwareInterface>hardware_interface/$(arg motors_controller_type)</hardwareInterface>
             <mechanicalReduction>1</mechanicalReduction>
          </actuator>
       </transmission>
-      <transmission name="wheel2_joint_transmission">
-         <type>transmission_interface/SimpleTransmission</type>
-         <joint name="wheel2_joint">
-            <hardwareInterface>hardware_interface/$(arg motors_controller_type)</hardwareInterface>
-         </joint>
-         <actuator name="wheel2_joint_actuator">
-            <hardwareInterface>hardware_interface/$(arg motors_controller_type)</hardwareInterface>
-            <mechanicalReduction>1</mechanicalReduction>
-         </actuator>
-      </transmission>
-      <transmission name="wheel3_joint_transmission">
-         <type>transmission_interface/SimpleTransmission</type>
-         <joint name="wheel3_joint">
-            <hardwareInterface>hardware_interface/$(arg motors_controller_type)</hardwareInterface>
-         </joint>
-         <actuator name="wheel3_joint_actuator">
-            <hardwareInterface>hardware_interface/$(arg motors_controller_type)</hardwareInterface>
-            <mechanicalReduction>1</mechanicalReduction>
-         </actuator>
-      </transmission>
-<!-- subwheels transmission links: required for tf-->
-<xacro:macro name="transmission_subwheel_macro" params="pos orient">
-<transmission name="subwheel${pos}_${orient}_joint_transmission">
-   <type>transmission_interface/SimpleTransmission</type>
-   <joint name="subwheel${pos}_${orient}_joint">
-      <hardwareInterface>hardware_interface/$(arg motors_controller_type)</hardwareInterface>
-   </joint>
-   <actuator name="subwheel${pos}_${orient}_joint_actuator">
-      <hardwareInterface>hardware_interface/$(arg motors_controller_type)</hardwareInterface>
-      <mechanicalReduction>1</mechanicalReduction>
-   </actuator>
-</transmission>
-</xacro:macro>
-<xacro:macro name="transmission_subwheel_pos_macro" params="pos">
-<xacro:transmission_subwheel_macro pos="${pos}" orient="top">
-</xacro:transmission_subwheel_macro>
-<xacro:transmission_subwheel_macro pos="${pos}" orient="left">
-</xacro:transmission_subwheel_macro>
-<xacro:transmission_subwheel_macro pos="${pos}" orient="right">
-</xacro:transmission_subwheel_macro>
-<xacro:transmission_subwheel_macro pos="${pos}" orient="bottom">
-</xacro:transmission_subwheel_macro>
-</xacro:macro>
-<!-- subwheels transmission's are not required or? (In case you  are not interested in the tf's of them -->
-<!-- generate subwheel transmission links: -->
-<!--<xacro:transmission_subwheel_pos_macro pos="1">
-</xacro:transmission_subwheel_pos_macro>
-<xacro:transmission_subwheel_pos_macro pos="2">
-</xacro:transmission_subwheel_pos_macro>
-<xacro:transmission_subwheel_pos_macro pos="3">
-</xacro:transmission_subwheel_pos_macro>-->
-  <!-- </xacro:unless>-->
-  <!-- p3d plugin (3D Position Interface for Ground Truth) -->
-  <xacro:if value="$(arg ground_truth)">
-    <gazebo>
-      <plugin name="ground_truth" filename="libgazebo_ros_p3d.so">
-        <frameName>world</frameName>
-        <bodyName>base_footprint</bodyName>
-        <topicName>/gazebo/$(arg robot_name)/odom</topicName>
-        <updateRate>100.0</updateRate>
-      </plugin>
-    </gazebo>
-  </xacro:if>
+   </xacro:macro>
+   <xacro:macro name="transmission_subwheel_pos_macro" params="pos">
+      <xacro:transmission_subwheel_macro pos="${pos}" orient="1_in" />
+      <xacro:transmission_subwheel_macro pos="${pos}" orient="2_in" />
+      <xacro:transmission_subwheel_macro pos="${pos}" orient="3_in" />
+      <xacro:transmission_subwheel_macro pos="${pos}" orient="4_in" />
+      <xacro:transmission_subwheel_macro pos="${pos}" orient="5_in" />
+      <xacro:transmission_subwheel_macro pos="${pos}" orient="1_out" />
+      <xacro:transmission_subwheel_macro pos="${pos}" orient="2_out" />
+      <xacro:transmission_subwheel_macro pos="${pos}" orient="3_out" />
+      <xacro:transmission_subwheel_macro pos="${pos}" orient="4_out" />
+      <xacro:transmission_subwheel_macro pos="${pos}" orient="5_out" />
+   </xacro:macro>
+   <!-- subwheels transmission's are not required or?
+   In case you  are not interested in the tf's of them visualized in rviz gnerate them!-->
+   <!-- generate subwheel transmission links: -->
+   <xacro:transmission_subwheel_pos_macro pos="1">
+   </xacro:transmission_subwheel_pos_macro>
+   <xacro:transmission_subwheel_pos_macro pos="2">
+   </xacro:transmission_subwheel_pos_macro>
+   <xacro:transmission_subwheel_pos_macro pos="3">
+   </xacro:transmission_subwheel_pos_macro>
+   <!-- p3d plugin (3D Position Interface for Ground Truth) -->
+   <xacro:if value="$(arg ground_truth)">
+      <gazebo>
+         <plugin name="ground_truth" filename="libgazebo_ros_p3d.so">
+            <frameName>world</frameName>
+            <bodyName>base_footprint</bodyName>
+            <topicName>/gazebo/$(arg robot_name)/odom</topicName>
+            <updateRate>10.0</updateRate> <!-- not sure why but if you set this value low ball is not so often jumping into the origin (in rviz) -->
+         </plugin>
+      </gazebo>
+   </xacro:if>
    <!-- links: http://gazebosim.org/tutorials/?tut=ros_urdf-->
    <!--no multiple physics engines through urdf?!  -->
@@ -101,5 +106,5 @@
       <maxVel>0.01</maxVel>
       <minDepth>0</minDepth>
-      <mu1>0.0</mu1> <!-- das ist die Reibung am Boden oder?! -->
+      <mu1>0.0</mu1>
       <mu2>0.0</mu2>
       <fdir1>0 0 0</fdir1>
@@ -111,117 +116,113 @@
       <material>Gazebo/DarkGrey</material>
    </gazebo>
-<!--  <gazebo reference="camera_mount_link">
+   <!--  <gazebo reference="camera_mount_link">
       <material>Gazebo/DarkGrey</material>
   </gazebo>-->
-<!-- main wheels:
+<!-- do i need this for ground friction?! -->
+<gazebo reference="base_footprint">
+   <mu1>1000</mu1>
+   <mu2>1000</mu2>
+   <material>Gazebo/Green</material>
+</gazebo>
+   <!-- main wheels:
 mu: Friction coefficients μ for the principal contact directions along the contact surface
-kp: Contact stiffness for rigid body contacts
+kp: Contact stiffness for rigid body contacts  (Steifigkeit)
 kd: Contact damping k_d for rigid body contacts
 mu of speichen_wheel actually does not matter cause it has no contact point!
 -->
-<xacro:macro name="wheel" params="pos">
-<gazebo reference="wheel${pos}_link">
-<mu1>0</mu1>
-<mu2>0</mu2>
-<kp>500000.0</kp>
-<kd>10.0</kd>
-<minDepth>0.001</minDepth>
-<maxVel>0.1</maxVel>
-<fdir1>1 0 0</fdir1>
-<material>Gazebo/Grey</material>
-</gazebo>
-</xacro:macro>
-<!-- generate wheels: -->
-<xacro:wheel pos="1"> </xacro:wheel>
-<xacro:wheel pos="2"> </xacro:wheel>
-<xacro:wheel pos="3"> </xacro:wheel>
-<!-- subwheels: -->
-<xacro:macro name="subwheel_params" params="suffix">
-<gazebo reference="subwheel${suffix}_link">
-<mu1>0.5</mu1>
-<mu2>0.5</mu2>
-<kp>500000.0</kp>
-<kd>100.0</kd>
-<minDepth>0.001</minDepth>
-<maxVel>0.1</maxVel>
-<fdir1>1 0 0</fdir1>
-<material>Gazebo/DarkGrey</material>
-</gazebo>
-</xacro:macro>
-<xacro:macro name="subwheel" params="pos">
-<xacro:subwheel_params suffix="${pos}_1_out">
-</xacro:subwheel_params>
-<xacro:subwheel_params suffix="${pos}_2_out">
-</xacro:subwheel_params>
-<xacro:subwheel_params suffix="${pos}_3_out">
-</xacro:subwheel_params>
-<xacro:subwheel_params suffix="${pos}_4_out">
-</xacro:subwheel_params>
-<xacro:subwheel_params suffix="${pos}_5_out">
-</xacro:subwheel_params>
-<xacro:subwheel_params suffix="${pos}_1_in">
-</xacro:subwheel_params>
-<xacro:subwheel_params suffix="${pos}_2_in">
-</xacro:subwheel_params>
-<xacro:subwheel_params suffix="${pos}_3_in">
-</xacro:subwheel_params>
-<xacro:subwheel_params suffix="${pos}_4_in">
-</xacro:subwheel_params>
-<xacro:subwheel_params suffix="${pos}_5_in">
-</xacro:subwheel_params>
-</xacro:macro>
-<!-- generate subwheels -->
-<xacro:subwheel pos="1"> </xacro:subwheel>
-<xacro:subwheel pos="2"> </xacro:subwheel>
-<xacro:subwheel pos="3"> </xacro:subwheel>
+   <xacro:macro name="wheel" params="pos">
+      <gazebo reference="wheel${pos}_link">
+         <mu1>0</mu1>
+         <mu2>0</mu2>
+         <kp>1e+13</kp>
+         <kd>1.0</kd>
+         <minDepth>0.001</minDepth>
+         <maxVel>0.1</maxVel>
+         <fdir1>1 0 0</fdir1>
+         <material>Gazebo/Grey</material>
+      </gazebo>
+   </xacro:macro>
+   <!-- generate wheels: -->
+   <xacro:wheel pos="1" />
+   <xacro:wheel pos="2" />
+   <xacro:wheel pos="3" />
+   <!-- subwheels: -->
+   <xacro:macro name="subwheel_params" params="suffix">
+      <gazebo reference="subwheel${suffix}_link">
+         <mu1>1000</mu1>
+         <mu2>1000</mu2>
+         <kp>5e+5</kp>
+         <kd>10.0</kd>
+         <minDepth>0.001</minDepth>
+         <maxVel>0.1</maxVel>
+         <fdir1>1 0 0</fdir1>
+         <material>Gazebo/DarkGrey</material>
+      </gazebo>
+   </xacro:macro>
+   <xacro:macro name="subwheel" params="pos">
+      <xacro:subwheel_params suffix="${pos}_1_out" />
+      <xacro:subwheel_params suffix="${pos}_2_out" />
+      <xacro:subwheel_params suffix="${pos}_3_out" />
+      <xacro:subwheel_params suffix="${pos}_4_out" />
+      <xacro:subwheel_params suffix="${pos}_5_out" />
+      <xacro:subwheel_params suffix="${pos}_1_in" />
+      <xacro:subwheel_params suffix="${pos}_2_in" />
+      <xacro:subwheel_params suffix="${pos}_3_in" />
+      <xacro:subwheel_params suffix="${pos}_4_in" />
+      <xacro:subwheel_params suffix="${pos}_5_in" />
+   </xacro:macro>
+   <!-- generate subwheels -->
+   <xacro:subwheel pos="1" />
+   <xacro:subwheel pos="2" />
+   <xacro:subwheel pos="3" />
    <!-- sensor links here! -->
-<gazebo reference="imu_link">
-  <sensor name="imu" type="imu">
-    <imu/>
-    <plugin filename="libgazebo_ros_imu_sensor.so" name="imu_plugin">
-      <robotNamespace/>
-      <frameName>imu_link</frameName>
-      <topicName>/$(arg robot_name)/sensor/imu</topicName>
-      <updateRateHZ>100.0</updateRateHZ>
-      <gaussianNoise>0.001</gaussianNoise>
-      <xyzOffset>0.0 0.0 0.0</xyzOffset>
-      <rpyOffset>0.0 0.0 0.0</rpyOffset>
-    </plugin>
-  </sensor>
-</gazebo>
-<gazebo reference="base_scan">
-   <material>Gazebo/Yellow</material>
-   <sensor name="lds_lfcd_sensor" type="ray">
-     <pose>0 0 0 0 0 0</pose>
-     <visualize>False</visualize>
-     <update_rate>5</update_rate>
-     <ray>
-       <scan>
-         <horizontal>
-           <samples>360</samples>
-           <resolution>1</resolution>
-           <min_angle>0.0</min_angle>
-           <max_angle>6.28</max_angle>
-         </horizontal>
-       </scan>
-       <range>
-         <min>0.120</min>
-         <max>3.5</max>
-         <resolution>0.015</resolution>
-       </range>
-       <noise>
-         <type>gaussian</type>
-         <mean>0.0</mean>
-         <stddev>0.01</stddev>
-       </noise>
-     </ray>
-     <plugin filename="libgazebo_ros_laser.so" name="gazebo_ros_lds_lfcd_controller">
-       <robotNamespace>/$(arg robot_name)/sensor</robotNamespace>
-       <topicName>scan_raw</topicName>
-       <frameName>base_scan</frameName>
-     </plugin>
-   </sensor>
- </gazebo>
-<!-- real sense stuff in realsense_camera.urdf.xacro -->
-  <!-- https://answers.ros.org/question/12430/modelling-sensorsimu-in-gazebo/ libgazebo_ros_imu.so-->
+   <gazebo reference="imu_link">
+      <sensor name="imu" type="imu">
+         <imu />
+         <plugin filename="libgazebo_ros_imu_sensor.so" name="imu_plugin">
+            <robotNamespace />
+            <frameName>imu_link</frameName>
+            <topicName>/$(arg robot_name)/sensor/imu</topicName>
+            <updateRateHZ>$(arg imu_update_rate)</updateRateHZ>
+            <gaussianNoise>0.00</gaussianNoise> <!-- was before: 0.001 -->
+            <xyzOffset>0.0 0.0 0.0</xyzOffset>
+            <rpyOffset>0.0 0.0 0.0</rpyOffset>
+         </plugin>
+      </sensor>
+   </gazebo>
+   <gazebo reference="base_scan">
+      <material>Gazebo/Yellow</material>
+      <sensor name="lds_lfcd_sensor" type="ray">
+         <pose>0 0 0 0 0 0</pose>
+         <visualize>False</visualize>
+         <update_rate>5</update_rate>
+         <ray>
+            <scan>
+               <horizontal>
+                  <samples>360</samples>
+                  <resolution>1</resolution>
+                  <min_angle>0.0</min_angle>
+                  <max_angle>6.28</max_angle>
+               </horizontal>
+            </scan>
+            <range>
+               <min>0.120</min>
+               <max>3.5</max>
+               <resolution>0.015</resolution>
+            </range>
+            <noise>
+               <type>gaussian</type>
+               <mean>0.0</mean>
+               <stddev>0.01</stddev>
+            </noise>
+         </ray>
+         <plugin filename="libgazebo_ros_laser.so" name="gazebo_ros_lds_lfcd_controller">
+            <robotNamespace>/$(arg robot_name)/sensor</robotNamespace>
+            <topicName>scan_raw</topicName>
+            <frameName>base_scan</frameName>
+         </plugin>
+      </sensor>
+   </gazebo>
+   <!-- real sense stuff in realsense_camera.urdf.xacro -->
+   <!-- https://answers.ros.org/question/12430/modelling-sensorsimu-in-gazebo/ libgazebo_ros_imu.so-->
 </robot>

Commit message: update docu pics

File: src/ballbot/bb_descrpition/urdf/ball_double_wheel.gazebo.xacro (robot description, xacro)
@@ -5,8 +5,8 @@
       <maxVel>0.01</maxVel>
       <minDepth>0</minDepth>
-      <mu1>1000</mu1>
-      <mu2>1000</mu2>
+      <mu1>1e+3</mu1>
+      <mu2>1e+3</mu2>
       <fdir1>0 0 0</fdir1>
-      <kp>5e+6</kp>
+      <kp>5e+5</kp>
       <kd>10.0</kd>
       <selfCollide>0</selfCollide>

File: src/ballbot/bb_descrpition/urdf/bb.urdf_double_wheel.xacro (robot description, xacro)
@@ -18,5 +18,5 @@
    <!-- subwheels parameters : -->
    <xacro:property name="mass_subwheel" value="0.006" />
-   <xacro:property name="d_inertia_subwheel" value="0.00000001" />    <!-- unit is kg m^2 diagonal inertia value for ixx,iyy,izz -->
+   <xacro:property name="d_inertia_subwheel" value="1e-8" />    <!-- unit is kg m^2 diagonal inertia value for ixx,iyy,izz -->
    <!--motor values:-->
    <!-- calculate max effort with emanual: http://support.robotis.com/en/product/actuator/dynamixel_x/xm_series/xm430-w350.htm -->
@@ -115,5 +115,5 @@
             <xacro:insert_block name="joint_origin_sub" />
             <axis xyz="1 0 0" />
-            <limit effort="0" velocity="0" />
+            <limit effort="0.0" velocity="0.0" />
             <dynamics friction="0.0" damping="0.0" />
          </joint>

File: src/ballbot/bb_descrpition/urdf/bb_double_wheel.gazebo.xacro (robot description, xacro)
@@ -122,6 +122,6 @@
 <!-- do i need this for ground friction?! -->
 <gazebo reference="base_footprint">
-   <mu1>1000</mu1>
-   <mu2>1000</mu2>
+   <mu1>1e+3</mu1>
+   <mu2>1e+3</mu2>
    <material>Gazebo/Green</material>
 </gazebo>
@@ -151,6 +151,6 @@
    <xacro:macro name="subwheel_params" params="suffix">
       <gazebo reference="subwheel${suffix}_link">
-         <mu1>1000</mu1>
-         <mu2>1000</mu2>
+         <mu1>1e+3</mu1>
+         <mu2>1e+3</mu2>
          <kp>5e+5</kp>
          <kd>10.0</kd>

Commit message: changed Kp, kd of ball now balancing up to 90sec

File: src/ballbot/bb_descrpition/urdf/ball_double_wheel.gazebo.xacro (robot description, xacro)
@@ -8,6 +8,6 @@
       <mu2>1e+3</mu2>
       <fdir1>0 0 0</fdir1>
-      <kp>5e+5</kp>
-      <kd>10.0</kd>
+      <kp>1e+18</kp>
+      <kd>1.0</kd>
       <selfCollide>0</selfCollide>
       <maxContacts>10</maxContacts>

File: src/ballbot/bb_descrpition/urdf/bb.urdf_double_wheel.xacro (robot description, xacro)
@@ -7,5 +7,7 @@
    <xacro:include filename="$(find ballbot_description)/urdf/common_properties.xacro" />
    <xacro:include filename="$(find ballbot_description)/urdf/bb_double_wheel.gazebo.xacro" />
+   <xacro:if value="$(arg use_realsense)">
    <xacro:include filename="$(find ballbot_description)/urdf/realsense_camera.urdf.xacro" />
+   </xacro:if>
    <!--<xacro:include filename="$(find hector_xacro_tools)/urdf/inertia_tensors.urdf.xacro" />-->
    <!-- some properties:
@@ -51,5 +53,5 @@
          <inertial>
             <origin xyz="0.0 0.0 0.05" /> <!-- important: here you can set the center of mass position! -->
-            <mass value="1.572" />             <!-- eigentlich: ixx="0.1" ixy="0.001" ixz="0.002" iyy="0.099" iyz="0.00" izz="0.007" -->
+            <mass value="1.572" /> <!-- eig. 1.572 -->  <!-- eigentlich: ixx="0.1" ixy="0.001" ixz="0.002" iyy="0.099" iyz="0.00" izz="0.007" -->
             <inertia ixx="0.1" ixy="0.00" ixz="0.00" iyy="0.1" iyz="0.00" izz="0.007" />
          </inertial>
@@ -190,4 +192,5 @@
       </link>
       <!--laser sensor: -->
+      <xacro:if value="$(arg use_laser)">
       <joint name="scan_joint" type="fixed">
          <parent link="body_link" />
@@ -217,4 +220,6 @@
   </inertial>
 </link>
+</xacro:if>
+<xacro:if value="$(arg use_realsense)">
 <joint name="realsense_mount_joint" type="fixed">
 <parent link="body_link" />
@@ -248,4 +253,5 @@
   <origin xyz="0.0 0.005 -0.00337" rpy="0.0 0.0 ${pi}" />
 </xacro:realsense_camera>
+   </xacro:if> <!-- end realsense -->
    </xacro:macro>
 </robot>

File: src/ballbot/bb_descrpition/urdf/bb_double_wheel.gazebo.xacro (robot description, xacro)
@@ -5,8 +5,9 @@
    <xacro:arg name="control_period" default="0.01" />
    <xacro:arg name="laser_visual" default="False" /> <!-- If this is true only in gazebo the lds scanner is visualized in blue! -->
-   <xacro:arg name="ground_truth" default="False" />
-    <!-- not used yet: -->
+   <xacro:arg name="ground_truth" default="True" />
+   <xacro:arg name="use_laser" default="True"/>
+   <xacro:arg name="use_realsense" default="True"/>
+   <!-- not used yet: -->
    <xacro:arg name="imu_visual" default="False" />
-   <xacro:arg name="use_diff_drive" default="False" />
    <!-- controllers: -->
    <gazebo>
@@ -192,4 +193,5 @@
       </sensor>
    </gazebo>
+<xacro:if value="$(arg use_laser)">
 <gazebo reference="base_scan">
   <material>Gazebo/DarkGrey</material>
@@ -225,4 +227,5 @@
   </sensor>
 </gazebo>
+</xacro:if>
    <!-- real sense stuff in realsense_camera.urdf.xacro -->
    <!-- https://answers.ros.org/question/12430/modelling-sensorsimu-in-gazebo/ libgazebo_ros_imu.so-->
