Commit message: balancing up to 2min

File: src/ballbot/bb_descrpition/urdf/ball_double_wheel.gazebo.xacro (robot description, xacro)
@@ -8,5 +8,5 @@
       <mu2>1e+3</mu2>
       <fdir1>0 0 0</fdir1>
-      <kp>1e+18</kp>
+      <kp>1e+15</kp>
       <kd>1.0</kd>
       <selfCollide>0</selfCollide>

File: src/ballbot/bb_descrpition/urdf/bb.urdf_double_wheel.xacro (robot description, xacro)
@@ -25,6 +25,6 @@
    <!-- dynamixel: XM430-W350-T: see performance graph the effort depends on current, efficiency(E), torque : -->
    <!-- http://simplemotor.com/calculations/ τ = (I * V * E *60) / (rpm * 2π) -->
-   <xacro:property name="XL430_W250_max_effort" value="4.1" />    <!-- sollte: 1.5 -> klappt damit aber nicht. nimm 4.1 -->
-   <xacro:property name="XL430_W250_max_velocity" value="5.7" />  <!-- sollte: ${61 * 2*pi/60}  klappt damit aber nicht nimm 5.7-->
+   <xacro:property name="XM430_W350_R_max_effort" value="3.8" />    <!-- acc. to datasheet should be 3.8Nm at 11.1V-->
+   <xacro:property name="XM430_W350_R_max_velocity" value="4.2" />  <!-- CAUTION set this param higher than 4 that the sim. works! for control mode max vel of this motors not specified! we measured: v_max=2 rad/sec;  -->
    <!-- trägheit des motors: if these values are higher than the torques wheel does not turn, if this value is not small enough gazebo error-->
    <!-- damping: is the damping force which is proportional to the velocity of the moving body [Nm*s/rad] -->
@@ -73,5 +73,5 @@
             <xacro:insert_block name="joint_origin" />
             <axis xyz="1 0 0" />
-            <limit effort="${XL430_W250_max_effort}" velocity="${XL430_W250_max_effort}" />
+            <limit effort="${XM430_W350_R_max_effort}" velocity="${XM430_W350_R_max_velocity}" />
             <dynamics friction="${wheel_joint_friction}" damping="${wheel_joint_damping}" />
          </joint>

File: src/ballbot/bb_descrpition/urdf/bb_double_wheel.gazebo.xacro (robot description, xacro)
@@ -154,6 +154,6 @@
          <mu1>1e+3</mu1>
          <mu2>1e+3</mu2>
-         <kp>5e+5</kp>
-         <kd>10.0</kd>
+         <kp>1e+10</kp>
+         <kd>1.0</kd>
          <minDepth>0.001</minDepth>
          <maxVel>0.1</maxVel>
