Commit message: update

File: src/ballbot/bb_descrpition/urdf/bb.urdf.xacro (robot description, xacro)
@@ -68,5 +68,5 @@
    <xacro:insert_block name="joint_origin" />
    <axis xyz="1 0 0" />
-   <limit effort="${XL430_W250_max_effort}" velocity="${XL430_W250_max_effort}" />
+   <limit effort="${XL430_W250_max_effort}" velocity="${XL430_W250_max_velocity}" />
    <dynamics friction="${wheel_joint_friction}" damping="${wheel_joint_damping}" />
 </joint>

File: src/ballbot/bb_descrpition/urdf/bb.urdf_double_wheel.xacro (robot description, xacro)
@@ -26,5 +26,5 @@
    <!-- http://simplemotor.com/calculations/ τ = (I * V * E *60) / (rpm * 2π) -->
    <xacro:property name="XM430_W350_R_max_effort" value="3.8" />    <!-- acc. to datasheet should be 3.8Nm at 11.1V-->
-   <xacro:property name="XM430_W350_R_max_velocity" value="4.2" />  <!-- CAUTION set this param higher than 4 that the sim. works! for control mode max vel of this motors not specified! we measured: v_max=2 rad/sec;  -->
+   <xacro:property name="XM430_W350_R_max_velocity" value="4.5" />  <!-- CAUTION set this param higher than 4 that the sim. works! for control mode max vel of this motors not specified! we measured: v_max=2 rad/sec;  -->
    <!-- trägheit des motors: if these values are higher than the torques wheel does not turn, if this value is not small enough gazebo error-->
    <!-- damping: is the damping force which is proportional to the velocity of the moving body [Nm*s/rad] -->

File: src/ballbot/bb_descrpition/urdf/bb_double_wheel.gazebo.xacro (robot description, xacro)
@@ -81,5 +81,5 @@
    <!-- subwheels transmission's are not required or?
    In case you  are not interested in the tf's of them visualized in rviz gnerate them!-->
-   <!-- generate subwheel transmission links: -->
+   <!-- generate subwheel transmission links:
    <xacro:transmission_subwheel_pos_macro pos="1">
    </xacro:transmission_subwheel_pos_macro>
@@ -88,4 +88,5 @@
    <xacro:transmission_subwheel_pos_macro pos="3">
    </xacro:transmission_subwheel_pos_macro>
+-->
    <!-- p3d plugin (3D Position Interface for Ground Truth) -->
    <xacro:if value="$(arg ground_truth)">
